File: kb-lone.kicad_pcb (KiCad board)
At the start: 2 copper layers, 304.8 x 114.3 mm, 475 parts, among them J1 TYPE-C-31-M12, J2 SM04B-SRSS-TB(LF)(SN), J3 SM04B-SRSS-TB(LF)(SN), J4 SSD1306, M1 RGB DB notch, Q1 DTC123JKAT146, SW1 K2-1187SQ-A4SW-06, SW10 F8, SW11 F9, SW12 F10, SW13 F11, SW14 F12, SW15 KNOB, SW16 GRV, SW17 1, SW18 2, SW19 3, SW2 ESC, SW20 4, SW21 5, SW22 6, SW23 7, SW24 8, SW25 9, SW26 0, SW27 MINUS, SW28 EQUAL, SW29 BSPC, SW3 F1, SW30 N/A, SW31 TAB, SW32 Q, SW33 W, SW34 E, SW35 R, SW36 T, SW37 Y, SW38 U, SW39 I, SW4 F2, SW40 O, SW41 P, SW42 LBRKT, SW43 RBRKT, SW44 BSLS, SW45 N/A, SW46 CAPS, SW47 A, SW48 S, SW49 D, SW5 F3, SW50 F, SW51 G, SW52 H, SW53 J, SW54 K, SW55 L, SW56 COLON, SW57 QUOTE, SW58 ENTER, SW59 PGUP, SW6 F4, SW60 LSHFT, SW61 Z, SW62 X, SW63 C, SW64 V, SW65 B, SW66 N, SW67 M, SW68 COMMA, SW69 DOT, SW7 F5, SW70 SLSH, SW71 RSHFT, SW72 UP, SW73 PGDN, SW74 LCTRL, SW75 WIN, SW76 LALT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

Commit message: place components
Parts:
- removed D16: 1N4148W, acheron_Components:D_SOD-123
- removed SW15: KNOB, acheron_MXH_MetalRings:MX100H
- removed X4: EXTRA_PINS, acheron_Connectors:PinHeader_2x3_P2.54mm_Vertical_Staggered
- J1, J4, SW84: moved to B.Cu
- moved U5 563.4 mm to (73.4, 57.5), turned to 90 degrees
- moved R96 561.7 mm to (56.0, 164.9), turned to 90 degrees
- moved U1 541.1 mm to (94.5, 62.3)
- moved R42 538.5 mm to (84.5, 89.7), turned to -90 degrees
- moved D46 518.1 mm to (71.4, 105.8), turned to 90 degrees
- moved C74 500.7 mm to (119.2, 127.8), turned to -90 degrees
- moved R57 490.9 mm to (91.6, 107.2), turned to -90 degrees
- moved C32 481.8 mm to (66.5, 69.0), turned to -90 degrees
- moved F1 468.6 mm to (99.7, 254.9)
- moved R54 468.3 mm to (153.5, 107.2), turned to -90 degrees
- moved SW84 467.0 mm to (54.4, 66.8)
- moved C3 462.4 mm to (60.4, 212.5)
- moved C5 462.4 mm to (60.4, 209.5)
- moved R13 462.4 mm to (74.7, 222.1)
- moved C13 462.4 mm to (127.0, 199.7)
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Routing:
- net C0: track 0.00 -> 113.5 mm
- net C14: track 0.00 -> 88.6 mm
- net Net-(D59-Pad2): track 0.00 -> 17.0 mm
- net Net-(D30-Pad2): track 0.00 -> 13.5 mm
- net Net-(D72-Pad2): track 0.00 -> 11.1 mm
- net Net-(D45-Pad2): track 0.00 -> 10.1 mm
- net Net-(D78-Pad2): track 0.00 -> 8.91 mm
- net Net-(D77-Pad2): track 0.00 -> 7.93 mm
- net Net-(D76-Pad2): track 0.00 -> 6.89 mm
- net Net-(D46-Pad2): track 0.00 -> 5.23 mm
- net Net-(D42-Pad2): track 0.00 -> 5.23 mm
- net Net-(D40-Pad2): track 0.00 -> 5.23 mm
- net Net-(D37-Pad2): track 0.00 -> 5.23 mm
- net Net-(D63-Pad2): track 0.00 -> 5.23 mm
- net Net-(D73-Pad2): track 0.00 -> 5.23 mm
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
Commit message: routing
Parts:
- added D16: 1N4148W, acheron_Components:D_SOD-123, F.Cu at (70.2, 67.7)
- added SW15: KNOB, acheron_MXA:MXA100, F.Cu at (61.9, 64.3)
- moved H7 171.1 mm to (281.1, 217.0)
- moved R13 156.0 mm to (91.9, 67.0)
- moved FB2 143.1 mm to (100.9, 66.6)
- moved H9 131.3 mm to (306.5, 208.3)
- moved Y1 109.4 mm to (152.8, 192.1)
- moved C9 90.3 mm to (178.8, 193.5)
- moved C3 70.8 mm to (128.4, 192.8)
- moved C5 70.8 mm to (128.4, 189.8)
- moved R10 70.8 mm to (136.8, 202.2)
- moved R9 70.8 mm to (139.7, 202.2)
- moved FB1 70.8 mm to (128.4, 186.9)
- moved M1 70.5 mm to (177.3, 213.9)
- moved F1 70.5 mm to (161.7, 221.2)
- moved C13 64.0 mm to (187.7, 179.5)
- moved R7 56.6 mm to (263.1, 180.9)
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Connections:
- U4 pad 10: E_PC2 -> C10
- U4 pad 11: E_PC3 -> C11
- U4 pad 14: E_PA0 -> C12
- U4 pad 15: E_PA1 -> C13
- U4 pad 16: E_PA2 -> C14
- U4 pad 20: R5 -> E_PA4
- U4 pad 21: R4 -> E_PA5
- U4 pad 22: R3 -> E_PA6
- U4 pad 23: C12 -> E_PA7
- U4 pad 24: C11 -> E_PC4
- U4 pad 25: C10 -> E_PC5
- U4 pad 26: C13 -> E_PB0
- U4 pad 27: C9 -> E_PB1
- U4 pad 29: C8 -> E_PB10
- U4 pad 33: C7 -> C0
- U4 pad 35: C6 -> C1
- U4 pad 37: C5 -> C2
- U4 pad 38: C4 -> C3
- U4 pad 39: C0 -> C4
- U4 pad 40: C1 -> C5
- U4 pad 41: C2 -> C6
- U4 pad 43: C3 -> C7
- U4 pad 50: E_PA14 -> R5
- U4 pad 51: E_PC10 -> R4
- U4 pad 52: C14 -> R3
- U4 pad 8: E_PC0 -> C8
- U4 pad 9: E_PC1 -> C9
- X3 pad 10: E_PA0 -> E_PC4
- X3 pad 11: E_PA1 -> E_PC5
- X3 pad 12: E_PA2 -> E_PB0
- X3 pad 13: E_PA3 -> E_PB1
- X3 pad 14: PA9 -> E_PB10
- X3 pad 5: E_PC0 -> E_PA3
- X3 pad 6: E_PC1 -> E_PA4
- X3 pad 7: E_PC2 -> E_PA5
- X3 pad 8: E_PC3 -> E_PA6
- X3 pad 9: E_PC10 -> E_PA7
Routing:
- net R1: track 0.00 -> 302.1 mm
- net R0: track 0.00 -> 299.1 mm
- net R2: track 0.00 -> 292.9 mm
- net R5: track 0.00 -> 286.2 mm
- net R3: track 0.00 -> 285.5 mm, vias 0 -> 1
- net R4: track 0.00 -> 274.9 mm
- net C12: track 0.00 -> 146.7 mm, vias 0 -> 6
- net C10: track 0.00 -> 142.4 mm, vias 0 -> 6
- net C11: track 0.00 -> 141.2 mm, vias 0 -> 6
- net C2: track 0.00 -> 136.9 mm, vias 0 -> 6
- net C1: track 0.00 -> 130.5 mm, vias 0 -> 5
- net C9: track 0.00 -> 129.2 mm, vias 0 -> 6
- net C4: track 0.00 -> 119.0 mm, vias 0 -> 6
- net C5: track 0.00 -> 113.9 mm, vias 0 -> 5
- net C6: track 0.00 -> 112.9 mm, vias 0 -> 6
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
Commit message: routing
Parts:
- removed X2: ARM JTAG, acheron_Connectors:PinHeader_2x5_P2.54mm_Vertical_Staggered
- removed X3: EXTRA_PINS, acheron_Connectors:PinHeader_1x16_P2.54mm_Vertical
- removed X5: Conn_01x03, acheron_Connectors:PinHeader_1x3_staggered_P2.54mm_Vertical
- R1, R2, U1: moved to B.Cu
- moved H9 255.0 mm to (98.1, 61.4)
- moved C18 229.6 mm to (60.2, 46.2)
- moved C17 223.6 mm to (66.2, 47.7)
- moved R14 218.8 mm to (71.0, 45.8)
- moved R13 208.9 mm to (272.9, 171.2)
- moved R1 193.7 mm to (87.1, 61.4), turned to 90 degrees
- moved R2 193.6 mm to (93.8, 61.4), turned to 90 degrees
- moved R4 171.1 mm to (352.4, 148.7)
- moved C1 163.6 mm to (353.8, 129.7)
- moved R3 142.7 mm to (353.8, 132.2), turned to 180 degrees
- moved D1 137.7 mm to (353.2, 145.9)
- moved R5 133.0 mm to (342.8, 149.9)
- moved R9 115.5 mm to (243.1, 150.7), turned to 180 degrees
- moved R10 115.2 mm to (239.8, 150.7)
- moved C8 90.4 mm to (262.0, 153.7)
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Connections:
- D101 pad 4: Net-(D100-Pad4) -> Net-(D100-Pad2)
- D125 pad 2: Net-(D125-Pad2) -> Net-(D124-Pad4)
- D125 pad 4: Net-(D124-Pad4) -> Net-(D125-Pad4)
- D126 pad 2: Net-(D126-Pad2) -> Net-(D125-Pad4)
- D126 pad 4: Net-(D125-Pad2) -> Net-(D126-Pad4)
- D127 pad 2: Net-(D127-Pad2) -> Net-(D126-Pad4)
- D127 pad 4: Net-(D126-Pad2) -> Net-(D127-Pad4)
- D128 pad 2: Net-(D113-Pad2) -> Net-(D127-Pad4)
- D128 pad 4: Net-(D127-Pad2) -> Net-(D113-Pad2)
- D137 pad 2: Net-(D137-Pad2) -> Net-(D138-Pad4)
- D138 pad 2: Net-(D137-Pad2) -> Net-(D138-Pad2)
- D139 pad 2: Net-(D138-Pad4) -> Net-(D139-Pad2)
- D139 pad 4: Net-(D139-Pad4) -> Net-(D138-Pad2)
- D140 pad 2: Net-(D139-Pad4) -> Net-(D140-Pad2)
- D140 pad 4: Net-(D140-Pad4) -> Net-(D139-Pad2)
- D141 pad 2: Net-(D140-Pad4) -> Net-(D141-Pad2)
- D141 pad 4: Net-(D141-Pad4) -> Net-(D140-Pad2)
- D142 pad 2: Net-(D141-Pad4) -> Net-(D142-Pad2)
- D142 pad 4: Net-(D142-Pad4) -> Net-(D141-Pad2)
- D153 pad 2: Net-(D153-Pad2) -> Net-(D152-Pad4)
- D153 pad 4: Net-(D152-Pad4) -> Net-(D153-Pad4)
- D154 pad 2: Net-(D154-Pad2) -> Net-(D153-Pad4)
- D154 pad 4: Net-(D153-Pad2) -> Net-(D154-Pad4)
- D155 pad 2: Net-(D155-Pad2) -> Net-(D154-Pad4)
- D155 pad 4: Net-(D154-Pad2) -> Net-(D155-Pad4)
- D156 pad 2: Net-(D142-Pad4) -> Net-(D155-Pad4)
- D156 pad 4: Net-(D155-Pad2) -> Net-(D142-Pad2)
- D157 pad 2: Net-(D143-Pad2) -> Net-(D157-Pad2)
- D157 pad 4: Net-(D157-Pad4) -> Net-(D143-Pad2)
- D158 pad 2: Net-(D157-Pad4) -> Net-(D158-Pad2)
- D158 pad 4: Net-(D158-Pad4) -> Net-(D157-Pad2)
- D159 pad 2: Net-(D158-Pad4) -> Net-(D159-Pad2)
- D159 pad 4: Net-(D159-Pad4) -> Net-(D158-Pad2)
- D160 pad 4: Net-(D159-Pad4) -> Net-(D159-Pad2)
- D99 pad 2: Net-(D85-Pad2) -> Net-(D100-Pad4)
- D99 pad 4: Net-(D100-Pad2) -> Net-(D85-Pad2)
- U4 pad 49: SWCLK -> ENC_SW
- U4 pad 50: R5 -> ENC_B
- U4 pad 51: R4 -> ENC_A
- U4 pad 52: R3 -> R5
- U4 pad 53: R2 -> R4
- U4 pad 54: R1 -> R3
- U4 pad 55: R0 -> R2
- U4 pad 56: E_PB4 -> R1
- U4 pad 57: ENC_A -> R0
- U4 pad 61: ENC_B -> E_PB8
- U4 pad 62: ENC_SW -> E_PB9
Routing:
- net Net-(D159-Pad2): track 0.00 -> 74.7 mm
- net Net-(D97-Pad4): track 0.00 -> 74.5 mm
- net Net-(D160-Pad2): track 0.00 -> 72.0 mm
- net 3V3: track 4.17 -> 64.9 mm, vias 0 -> 8
- net SCL: track 4.63 -> 47.6 mm
- net Net-(D143-Pad2): track 0.00 -> 35.8 mm
- net 5V: track 84.0 -> 119.6 mm, vias 82 -> 83
- net Net-(D113-Pad2): track 0.00 -> 31.0 mm
- net Net-(D142-Pad2): track 0.00 -> 30.8 mm
- net GNDPWR: track 0.00 -> 29.0 mm
- net SDA: track 7.81 -> 35.9 mm
- net Net-(D140-Pad2): track 0.00 -> 28.1 mm
- net Net-(D143-Pad4): track 0.00 -> 27.2 mm
- net Net-(D141-Pad2): track 0.00 -> 26.9 mm
- net Net-(D85-Pad2): track 0.00 -> 26.9 mm
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
Commit message: routing
Parts:
- moved H1 280.5 mm to (81.7, 61.5)
- moved C2 154.0 mm to (354.1, 140.7)
- moved FB1 127.5 mm to (81.7, 68.3), turned to -90 degrees
- moved R12 94.0 mm to (268.1, 157.8), turned to 90 degrees
- moved C3 93.5 mm to (213.6, 154.2), turned to 90 degrees
- moved H4 74.9 mm to (225.9, 206.1)
- moved C10 72.5 mm to (199.3, 153.4), turned to -90 degrees
- moved R11 69.0 mm to (270.9, 157.8), turned to 90 degrees
- moved M1 59.4 mm to (169.4, 155.0)
- moved Y1 57.3 mm to (197.7, 156.5)
- moved H3 54.6 mm to (254.0, 197.0)
- moved H5 54.6 mm to (237.7, 215.4)
- moved H8 54.6 mm to (243.6, 190.4)
- moved H2 54.6 mm to (245.6, 221.7)
- moved H6 54.6 mm to (239.7, 201.2)
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Connections:
- U4 pad 33: C0 -> E_PB12
- U4 pad 35: C1 -> C0
- U4 pad 36: RGB_3V3 -> C1
- U4 pad 61: E_PB8 -> RGB_3V3
Routing:
- net 3V3: track 64.9 -> 110.7 mm
- net ENC_B: track 4.55 -> 25.1 mm
- net Net-(R14-Pad2): track 0.00 -> 16.3 mm
- net ENC_A: track 5.37 -> 21.6 mm
- net SDA: track 35.9 -> 51.3 mm
- net BOOT0: track 7.43 -> 22.8 mm
- net C14: track 118.1 -> 132.3 mm
- net PA9: track 0.00 -> 12.6 mm
- net I2C_DAT: track 0.00 -> 10.7 mm, vias 0 -> 1
- net 5V: track 119.6 -> 129.1 mm, vias 83 -> 82
- net C4: track 119.0 -> 109.7 mm, vias 6 -> 5
- net Net-(D143-Pad2): track 35.8 -> 27.8 mm
- net D+: track 11.5 -> 19.4 mm
- net I2C_CLK: track 0.00 -> 6.83 mm, vias 0 -> 1
- net Net-(FB1-Pad1): track 0.00 -> 5.75 mm
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
Commit message: routing
Routing:
- net C6: track 112.9 -> 1057.1 mm, vias 6 -> 10
- net C5: track 109.7 -> 891.3 mm, vias 5 -> 10
- net C4: track 109.7 -> 743.2 mm, vias 5 -> 10
- net C3: track 109.8 -> 596.1 mm, vias 5 -> 10
- net C2: track 136.9 -> 450.2 mm, vias 6 -> 11
- net C1: track 130.5 -> 315.2 mm, vias 5 -> 10
- net C10: track 142.4 -> 64.4 mm, vias 6 -> 10
- net C9: track 129.2 -> 61.6 mm, vias 6 -> 10
- net C8: track 109.5 -> 57.9 mm, vias 5 -> 9
- net C7: track 109.5 -> 58.2 mm, vias 5 -> 9
- net ENC_A: track 21.6 -> 68.4 mm, vias 0 -> 1
- net C11: track 153.7 -> 124.8 mm, vias 6 -> 10
- net 5V: track 129.1 -> 156.9 mm
- net Net-(D85-Pad2): track 26.9 -> 0.00 mm
- net C12: track 146.7 -> 170.2 mm, vias 6 -> 7
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