File: kb-lone.kicad_pcb (KiCad board)
At the start: 2 copper layers, 304.8 x 114.3 mm, 471 parts, among them J1 TYPE-C-31-M12, J2 SM04B-SRSS-TB(LF)(SN), J3 SM04B-SRSS-TB(LF)(SN), J4 SSD1306, M1 RGB DB notch, Q1 DTC123JKAT146, SW1 K2-1187SQ-A4SW-06, SW10 F8, SW11 F9, SW12 F10, SW13 F11, SW14 F12, SW15 KNOB, SW16 GRV, SW17 1, SW18 2, SW19 3, SW2 ESC, SW20 4, SW21 5, SW22 6, SW23 7, SW24 8, SW25 9, SW26 0, SW27 MINUS, SW28 EQUAL, SW29 BSPC, SW3 F1, SW30 N/A, SW31 TAB, SW32 Q, SW33 W, SW34 E, SW35 R, SW36 T, SW37 Y, SW38 U, SW39 I, SW4 F2, SW40 O, SW41 P, SW42 LBRKT, SW43 RBRKT, SW44 BSLS, SW45 N/A, SW46 CAPS, SW47 A, SW48 S, SW49 D, SW5 F3, SW50 F, SW51 G, SW52 H, SW53 J, SW54 K, SW55 L, SW56 COLON, SW57 QUOTE, SW58 ENTER, SW59 PGUP, SW6 F4, SW60 LSHFT, SW61 Z, SW62 X, SW63 C, SW64 V, SW65 B, SW66 N, SW67 M, SW68 COMMA, SW69 DOT, SW7 F5, SW70 SLSH, SW71 RSHFT, SW72 UP, SW73 PGDN, SW74 LCTRL, SW75 WIN, SW76 LALT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

Commit message: routing
Parts:
- R1, R2, U1: moved to F.Cu
- moved M1 49.1 mm to (211.3, 180.5)
- moved R10 19.8 mm to (220.0, 149.5)
- moved R9 19.1 mm to (224.1, 149.5)
- moved R8 12.8 mm to (266.2, 166.0), turned to 0 degrees
- moved C16 4.42 mm to (262.6, 166.3)
- moved R12 3.76 mm to (265.2, 160.2), turned to 0 degrees
- moved C15 3.60 mm to (258.5, 166.4), turned to 0 degrees
- moved R13 3.43 mm to (262.7, 156.0), turned to 0 degrees
- moved J2 3.32 mm to (90.5, 66.1), turned to 0 degrees
- moved C14 3.19 mm to (246.5, 166.0)
- moved C6 3.02 mm to (246.1, 151.9), turned to 90 degrees
- moved R11 2.89 mm to (269.2, 160.1), turned to 0 degrees
- moved C7 2.37 mm to (243.5, 151.9), turned to 90 degrees
- moved C8 1.12 mm to (262.7, 154.5)
- moved C11 1.03 mm to (242.7, 161.3)
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Connections:
- D16 pad 2: Net-(D16-Pad2) -> ENC_SW
- SW15 pad 2: Net-(D16-Pad2) -> ENC_SW
- SW84 pad S2: GND -> ENC_SW
- U4 pad 10: C10 -> R2
- U4 pad 11: C11 -> R3
- U4 pad 14: C12 -> R4
- U4 pad 15: C13 -> R5
- U4 pad 52: R5 -> C8
- U4 pad 53: R4 -> C9
- U4 pad 54: R3 -> C10
- U4 pad 55: R2 -> C11
- U4 pad 56: R1 -> C12
- U4 pad 57: R0 -> C13
- U4 pad 8: C8 -> R0
- U4 pad 9: C9 -> R1
Routing:
- net C7: track 58.2 -> 838.7 mm
- net C8: track 57.9 -> 697.9 mm
- net C9: track 61.6 -> 575.0 mm, vias 10 -> 11
- net C10: track 64.4 -> 442.4 mm, vias 10 -> 11
- net C11: track 124.8 -> 295.5 mm, vias 10 -> 12
- net C0: track 208.9 -> 134.0 mm, vias 6 -> 1
- net ENC_SW: track 21.7 -> 87.4 mm, vias 1 -> 2
- net ENC_B: track 46.7 -> 98.8 mm, vias 1 -> 2
- net D-: track 11.5 -> 61.0 mm
- net D+: track 19.4 -> 60.5 mm
- net C2: track 450.2 -> 491.2 mm
- net ENC_A: track 68.4 -> 106.0 mm, vias 1 -> 2
- net E_PB0: track 0.00 -> 35.6 mm, vias 0 -> 1
- net E_PB1: track 0.00 -> 34.7 mm, vias 0 -> 1
- net E_PB10: track 0.00 -> 33.7 mm, vias 0 -> 1
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Other:
- outline, holes or cut-outs redrawn

Commit message: routing
Routing:
- net C6: track 1082.9 -> 368.6 mm
- net C5: track 907.9 -> 416.3 mm
- net C7: track 838.7 -> 351.0 mm
- net C4: track 759.7 -> 490.7 mm
- net C8: track 697.9 -> 433.7 mm
- net C9: track 575.0 -> 533.6 mm
- net C11: track 295.5 -> 274.5 mm
- net C10: track 442.4 -> 422.5 mm
- net C2: track 491.2 -> 499.3 mm
- net C3: track 612.7 -> 620.7 mm
- net C1: track 341.8 -> 349.0 mm
- net C12: track 195.4 -> 202.2 mm
