File: kb-lone.kicad_sch (KiCad schematic)
At the start: 495 parts, among them J1 TYPE-C-31-M12, J2 SM04B-SRSS-TB(LF)(SN), J3 SM04B-SRSS-TB(LF)(SN), J4 SSD1306, M1 RGB DB notch, Q1 DTC123JKAT146, SW1 K2-1187SQ-A4SW-06, SW10 CPG151101S11, SW11 CPG151101S11, SW12 CPG151101S11, SW13 CPG151101S11, SW14 CPG151101S11, SW15 CPG151101S11, SW16 CPG151101S11, SW17 CPG151101S11, SW18 CPG151101S11, SW19 CPG151101S11, SW2 CPG151101S11, SW20 CPG151101S11, SW21 CPG151101S11, SW22 CPG151101S11, SW23 CPG151101S11, SW24 CPG151101S11, SW25 CPG151101S11, SW26 CPG151101S11, SW27 CPG151101S11, SW28 CPG151101S11, SW29 CPG151101S11, SW3 CPG151101S11, SW30 CPG151101S11, SW31 CPG151101S11, SW32 CPG151101S11, SW33 CPG151101S11, SW34 CPG151101S11, SW35 CPG151101S11, SW36 CPG151101S11, SW37 CPG151101S11, SW38 CPG151101S11, SW39 CPG151101S11, SW4 CPG151101S11, SW40 CPG151101S11, SW41 CPG151101S11, SW42 CPG151101S11, SW43 CPG151101S11, SW44 CPG151101S11, SW45 CPG151101S11, SW46 CPG151101S11, SW47 CPG151101S11, SW48 CPG151101S11, SW49 CPG151101S11, SW5 CPG151101S11, SW50 CPG151101S11, SW51 CPG151101S11, SW52 CPG151101S11, SW53 CPG151101S11, SW54 CPG151101S11, SW55 CPG151101S11, SW56 CPG151101S11, SW57 CPG151101S11, SW58 CPG151101S11, SW59 CPG151101S11, SW6 CPG151101S11, SW60 CPG151101S11, SW61 CPG151101S11, SW62 CPG151101S11, SW63 CPG151101S11, SW64 CPG151101S11, SW65 CPG151101S11, SW66 CPG151101S11, SW67 CPG151101S11, SW68 CPG151101S11, SW69 CPG151101S11, SW7 CPG151101S11, SW70 CPG151101S11, SW71 CPG151101S11, SW72 CPG151101S11, SW73 CPG151101S11, SW74 CPG151101S11, SW75 CPG151101S11, SW76 CPG151101S11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

Commit message: schematics rgb leds
Parts:
- removed C101, C102, C103, C104, C65: 100n, apollo87h_kicad_library:C_0402_1005Metric_1, symbol Device:C_Small
- removed D138, D172, D173, D174, D175: SK6812MINI-E, acheron_Components:SK6812MINI_3535_6028_3.2x2.8mm_Round, symbol acheron_Symbols:SK6812MINI-E
- removed R100, R62, R97, R98, R99: 5.1R, apollo87h_kicad_library:R_0402_1005Metric_1, symbol Device:R_Small
- SW75: Keycode LGUI -> WIN
- renumbered C105 to C100, C67 to C17, C68 to C18, C17 to C33, C18 to C34, C33 to C35, C34 to C36, C35 to C37, C36 to C38, C37 to C39, C38 to C40, C39 to C41, C40 to C42, C41 to C43, C42 to C44, C43 to C45, C44 to C46, C45 to C47, C50 to C48, C51 to C49, C52 to C50, C53 to C51, C54 to C52, C55 to C53, C56 to C54, C57 to C55, C58 to C56, C59 to C57, C60 to C58, C46 to C59, C47 to C60, C48 to C61, C49 to C62, C69 to C63, C70 to C64, C71 to C65, C72 to C66, C73 to C67, C74 to C68, C75 to C69, C76 to C70, C77 to C71, C61 to C72, C62 to C73, C63 to C74, C64 to C75, C66 to C76, C85 to C77, C86 to C78, C87 to C79, C88 to C80, C89 to C81, C90 to C82, C91 to C83, C92 to C84, C93 to C85, C94 to C86, C78 to C87, C79 to C88, C80 to C89, C81 to C90, C82 to C91, C83 to C92, C84 to C93, C95 to C94, C96 to C95, C97 to C96, C98 to C97, C99 to C98, C100 to C99, D91 to D100, D106 to D101, D107 to D102, D108 to D103, D109 to D104, D110 to D105, D111 to D106, D112 to D107, D113 to D108, D114 to D109, D115 to D110, D116 to D111, D117 to D112, D118 to D113, D123 to D114, D124 to D115, D125 to D116, D126 to D117, D127 to D118, D128 to D119, D129 to D120, D130 to D121, D131 to D122, D132 to D123, D133 to D124, D119 to D125, D120 to D126, D121 to D127, D122 to D128, D140 to D129, D141 to D130, D142 to D131, D143 to D132, D144 to D133, D145 to D134, D146 to D135, D147 to D136, D148 to D137, D134 to D138, D135 to D139, D136 to D140, D137 to D141, D139 to D142, D156 to D143, D157 to D144, D158 to D145, D159 to D146, D160 to D147, D161 to D148, D162 to D149, D163 to D150, D164 to D151, D165 to D152, D149 to D153, D150 to D154, D151 to D155, D152 to D156, D153 to D157, D154 to D158, D155 to D159, D166 to D160, D167 to D161, D168 to D162, D169 to D163, D170 to D164, D171 to D165, D176 to D166, D92 to D85, D93 to D86, D94 to D87, D95 to D88, D96 to D89, D97 to D90, D98 to D91, D99 to D92, D100 to D93, D101 to D94, D102 to D95, D103 to D96, D104 to D97, D105 to D98, D90 to D99, R64 to R14, R16 to R15, R17 to R16, R18 to R17, R19 to R18, R20 to R19, R21 to R20, R22 to R21, R23 to R22, R24 to R23, R25 to R24, R26 to R25, R27 to R26, R28 to R27, R29 to R28, R14 to R29, R15 to R30, R30 to R31, R31 to R32, R32 to R33, R33 to R34, R34 to R35, R35 to R36, R36 to R37, R37 to R38, R38 to R39, R39 to R40, R40 to R41, R41 to R42, R42 to R43, R47 to R44, R48 to R45, R49 to R46, R50 to R47, R51 to R48, R52 to R49, R53 to R50, R54 to R51, R55 to R52, R56 to R53, R57 to R54, R43 to R55, R44 to R56, R45 to R57, R46 to R58, R65 to R59, R66 to R60, R67 to R61, R68 to R62, R69 to R63, R70 to R64, R71 to R65, R72 to R66, R73 to R67, R58 to R68, R59 to R69, R60 to R70, R61 to R71, R63 to R72, R81 to R73, R82 to R74, R83 to R75, R84 to R76, R85 to R77, R86 to R78, R87 to R79, R88 to R80, R89 to R81, R90 to R82, R74 to R83, R75 to R84, R76 to R85, R77 to R86, R78 to R87, R79 to R88, R80 to R89, R91 to R90, R92 to R91, R93 to R92, R94 to R93, R95 to R94, R96 to R95, R101 to R96
Connections:
- net E_PC15 is gone; now on net E_PC10: X3.9 (Pin_9)
- net E_PA0: now also X3.10 (Pin_10); no longer X3.14 (Pin_14)
- net E_PA1: now also X3.11 (Pin_11); no longer X3.15 (Pin_15)
- net E_PA14: now also X3.15 (Pin_15); no longer X4.4 (Pin_4)
- net E_PA2: now also X3.12 (Pin_12); no longer X3.16 (Pin_16)
- net E_PC0: now also X3.5 (Pin_5); no longer X3.10 (Pin_10)
- net E_PC1: now also X3.6 (Pin_6); no longer X3.11 (Pin_11)
- net E_PC10: no longer X4.6 (Pin_6)
- net E_PC13: now also X3.4 (Pin_4); no longer X3.7 (Pin_7)
- net E_PC2: now also X3.7 (Pin_7); no longer X3.12 (Pin_12)
- net E_PC3: now also X3.8 (Pin_8); no longer X3.13 (Pin_13)
- net GND: no longer C58.2
- net PA9: now also X3.14 (Pin_14); no longer X4.3 (Pin_3)
- net at D128.2 (DOUT): now also D113.2 (DOUT); no longer D142.4 (DIN)
- net I2C_CLK: now reaches J4.2 (SCL)
- net I2C_CLK: now also U4.4 (PC15/OSC32_OUT)
- net at D138.2 (DOUT): now also D137.2 (DOUT); no longer D124.4 (DIN)
- net at D165.2 (DOUT): now also D166.4 (DIN)
- net at D141.4 (DIN): now also D142.2 (DOUT)
- net at D157.2 (DOUT): now also D143.2 (DOUT); no longer D160.4 (DIN)
- net at D99.2 (DOUT): now also D85.2 (DOUT); no longer D101.4 (DIN)
- net at D159.4 (DIN): now also D160.4 (DIN); no longer D143.2 (DOUT)
- net at D100.4 (DIN): now also D101.4 (DIN); no longer D85.2 (DOUT)
- net at D125.4 (DIN): now also D124.4 (DIN); no longer D113.2 (DOUT)
- net E_PA3: now reaches U4.17 (PA3/TIM2_CH4/USART2_RX)
- net E_PA3: now also X3.13 (Pin_13)
- net E_PB4: now reaches U4.56 (NJTRST/SPI1_MISO/SPI3_MISO/I2C3_SDA/TIM3_CH1/PB4)
- net E_PB4: now also X3.16 (Pin_16)
- net at D153.4 (DIN): now also D152.4 (DIN); no longer D137.2 (DOUT)
- net at D156.2 (DOUT): now also D142.4 (DIN); no longer D152.4 (DIN)
- no-connect marks 4 -> 7
Other:
- note added: "BSLS"
- note added: "BSPC"
- note added: "CAPS"
- note added: "EQUAL"
- note added: "FN"
- note added: "KNOB"
- note added: "LALT"
- note added: "LBRKT"
- note added: "LCTRL"
- note added: "LSHFT"
- note added: "N/A"
- note added: "PG DN"
- note added: "PG UP"
- note added: "RALT"
- note added: "RBRKT"
- note added: "RCTRL"
- note added: "RGV"
- note added: "RSHFT"
- note added: "SLSH"
- note added: "WIN"
- note removed: "BACKSLASH"
- note removed: "BACKSPACE"
- note removed: "CAPS LOCK"
- note removed: "DELETE"
- note removed: "END"
- note removed: "FN2 MENU"
- note removed: "GRAVE"
- note removed: "HOME"
- note removed: "INSERT"
- note removed: "LEFT ALT"
- note removed: "LEFT BRACKET"
- note removed: "LEFT CONTROL"
- note removed: "LEFT GUI"
- note removed: "LEFT SHIFT"
- note removed: "PAGE DOWN"
- note removed: "PAGE UP"
- note removed: "PAUSE"
- note removed: "PLUS"
- note removed: "PRINT"
- note removed: "RIGHT ALT"
- note removed: "RIGHT BRACKET"
- note removed: "RIGHT CONTROL"
- note removed: "RIGHT GUI"
- note removed: "RIGHT SHIFT"
- note removed: "SCROLL LOCK"
- note removed: "SLASH"
- note removed: "SW5 was skipped to make firmware easier for the split right shift"
- note removed: "SW8 was skipped to make firmware easier for the ISO backslash"
- note removed: "SW8 was skipped to make firmware easier for the ISO tilde"
- moved on the sheet: C100, C19, C20, C21, C22, C23, C24, C25, C26, C27, C28, C29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

Commit message: place sw + rgb led
Parts:
- removed GR1: Apollo87H Logo, apollo87h_kicad_library:apollo87h_logo, symbol Mechanical:MountingHole
- removed GR2: Grounding sign, acheron_Graphics:grounding_sign_3.6x3.2mm, symbol Mechanical:MountingHole
- removed GR3: Acheron X Geon Logo, apollo87h_kicad_library:acheron_geon_logo_plated, symbol Mechanical:MountingHole
- removed GR4: Huge Apollo Logo, apollo87h_kicad_library:apollo_logo_120x120mm, symbol Mechanical:MountingHole
- removed GR5: Apollo Label, apollo87h_kicad_library:apollo87h_label, symbol Mechanical:MountingHole
- SW10: value CPG151101S11 -> F8; footprint acheron_MXH:MX100H -> acheron_MXH_MetalRings:MX100H
- SW11: value CPG151101S11 -> F9; footprint acheron_MXH:MX100H -> acheron_MXH_MetalRings:MX100H
- SW12: value CPG151101S11 -> F10; footprint acheron_MXH:MX100H -> acheron_MXH_MetalRings:MX100H
- SW13: value CPG151101S11 -> F11; footprint acheron_MXH:MX100H -> acheron_MXH_MetalRings:MX100H
- SW14: value CPG151101S11 -> F12; footprint acheron_MXH:MX100H -> acheron_MXH_MetalRings:MX100H
- SW15: value CPG151101S11 -> KNOB; footprint acheron_MXH:MX100H -> acheron_MXH_MetalRings:MX100H
- SW16: value CPG151101S11 -> GRV; footprint acheron_MXH:MX100H -> acheron_MXH_MetalRings:MX100H
- SW17: value CPG151101S11 -> 1; footprint acheron_MXH:MX100H -> acheron_MXH_MetalRings:MX100H
- SW18: value CPG151101S11 -> 2; footprint acheron_MXH:MX100H -> acheron_MXH_MetalRings:MX100H
- SW19: value CPG151101S11 -> 3; footprint acheron_MXH:MX100H -> acheron_MXH_MetalRings:MX100H
- SW2: value CPG151101S11 -> ESC; footprint acheron_MXH:MX100H -> acheron_MXH_MetalRings:MX100H
- SW20: value CPG151101S11 -> 4; footprint acheron_MXH:MX100H -> acheron_MXH_MetalRings:MX100H
- SW21: value CPG151101S11 -> 5; footprint acheron_MXH:MX100H -> acheron_MXH_MetalRings:MX100H
- SW22: value CPG151101S11 -> 6; footprint acheron_MXH:MX100H -> acheron_MXH_MetalRings:MX100H
- SW23: value CPG151101S11 -> 7; footprint acheron_MXH:MX100H -> acheron_MXH_MetalRings:MX100H
- SW24: value CPG151101S11 -> 8; footprint acheron_MXH:MX100H -> acheron_MXH_MetalRings:MX100H
- SW25: value CPG151101S11 -> 9; footprint acheron_MXH:MX100H -> acheron_MXH_MetalRings:MX100H
- SW26: value CPG151101S11 -> 0; footprint acheron_MXH:MX100H -> acheron_MXH_MetalRings:MX100H
- SW27: value CPG151101S11 -> MINUS; footprint acheron_MXH:MX100H -> acheron_MXH_MetalRings:MX100H
- SW28: value CPG151101S11 -> EQUAL; footprint acheron_MXH:MX100H -> acheron_MXH_MetalRings:MX100H
- SW29: value CPG151101S11 -> BSPC; footprint acheron_MXH:MX100H -> acheron_MXH_MetalRings:MX200H
- SW3: value CPG151101S11 -> F1; footprint acheron_MXH:MX100H -> acheron_MXH_MetalRings:MX100H
- SW30, SW45: value CPG151101S11 -> N/A; footprint acheron_MXH:MX100H -> acheron_MXH_MetalRings:MX100H
- SW31: value CPG151101S11 -> TAB; footprint acheron_MXH:MX200H -> acheron_MXH_MetalRings:MX150H
- SW32: value CPG151101S11 -> Q; footprint acheron_MXH:MX100H -> acheron_MXH_MetalRings:MX100H
- SW33: value CPG151101S11 -> W; footprint acheron_MXH:MX100H -> acheron_MXH_MetalRings:MX100H
- SW34: value CPG151101S11 -> E; footprint acheron_MXH:MX100H -> acheron_MXH_MetalRings:MX100H
- SW35: value CPG151101S11 -> R; footprint acheron_MXH:MX150H -> acheron_MXH_MetalRings:MX100H
- SW36: value CPG151101S11 -> T; footprint acheron_MXH:MX100H -> acheron_MXH_MetalRings:MX100H
- SW37: value CPG151101S11 -> Y; footprint acheron_MXH:MX100H -> acheron_MXH_MetalRings:MX100H
- SW38: value CPG151101S11 -> U; footprint acheron_MXH:MX100H -> acheron_MXH_MetalRings:MX100H
- SW39: value CPG151101S11 -> I; footprint acheron_MXH:MX100H -> acheron_MXH_MetalRings:MX100H
- SW4: value CPG151101S11 -> F2; footprint acheron_MXH:MX100H -> acheron_MXH_MetalRings:MX100H
- SW40: value CPG151101S11 -> O; footprint acheron_MXH:MX100H -> acheron_MXH_MetalRings:MX100H
- SW41: value CPG151101S11 -> P; footprint acheron_MXH:MX100H -> acheron_MXH_MetalRings:MX100H
- SW42: value CPG151101S11 -> LBRKT; footprint acheron_MXH:MX100H -> acheron_MXH_MetalRings:MX100H
- SW43: value CPG151101S11 -> RBRKT; footprint acheron_MXH:MX100H -> acheron_MXH_MetalRings:MX100H
- SW44: value CPG151101S11 -> BSLS; footprint acheron_MXH:MX100H -> acheron_MXH_MetalRings:MX150H
- SW46: value CPG151101S11 -> CAPS; footprint acheron_MXH:MX100H -> acheron_MXH_MetalRings:MX175H
- SW47: value CPG151101S11 -> A; footprint acheron_MXH:MX100H -> acheron_MXH_MetalRings:MX100H
- SW48: value CPG151101S11 -> S; footprint acheron_MXH:MX150H -> acheron_MXH_MetalRings:MX100H
- SW49: value CPG151101S11 -> D; footprint acheron_MXH:MX100H -> acheron_MXH_MetalRings:MX100H
- SW5: value CPG151101S11 -> F3; footprint acheron_MXH:MX100H -> acheron_MXH_MetalRings:MX100H
- SW50: value CPG151101S11 -> F; footprint acheron_MXH:MX100H -> acheron_MXH_MetalRings:MX100H
- SW51: value CPG151101S11 -> G; footprint acheron_MXH:MX100H -> acheron_MXH_MetalRings:MX100H
- SW52: value CPG151101S11 -> H; footprint acheron_MXH:MX175H -> acheron_MXH_MetalRings:MX100H
- SW53: value CPG151101S11 -> J; footprint acheron_MXH:MX100H -> acheron_MXH_MetalRings:MX100H
- SW54: value CPG151101S11 -> K; footprint acheron_MXH:MX100H -> acheron_MXH_MetalRings:MX100H
- SW55: value CPG151101S11 -> L; footprint acheron_MXH:MX100H -> acheron_MXH_MetalRings:MX100H
- SW56: value CPG151101S11 -> COLON; footprint acheron_MXH:MX100H -> acheron_MXH_MetalRings:MX100H
- SW57: value CPG151101S11 -> QUOTE; footprint acheron_MXH:MX100H -> acheron_MXH_MetalRings:MX100H
- SW58: value CPG151101S11 -> ENTER; footprint acheron_MXH:MX100H -> acheron_MXH_MetalRings:MX225HR
- SW59: value CPG151101S11 -> PGUP; footprint acheron_MXH:MX100H -> acheron_MXH_MetalRings:MX100H
- SW6: value CPG151101S11 -> F4; footprint acheron_MXH:MX100H -> acheron_MXH_MetalRings:MX100H
- SW60: value CPG151101S11 -> LSHFT; footprint acheron_MXH:MX100H -> acheron_MXH_MetalRings:MX225H; Keycode LSFT -> LSHFT
- SW61: value CPG151101S11 -> Z; footprint acheron_MXH:MX100H -> acheron_MXH_MetalRings:MX100H
- SW62: value CPG151101S11 -> X; footprint acheron_MXH:MX100H -> acheron_MXH_MetalRings:MX100H
- SW63: value CPG151101S11 -> C; footprint acheron_MXH:MX100H -> acheron_MXH_MetalRings:MX100H
- SW64: value CPG151101S11 -> V; footprint acheron_MXH:MX225HR -> acheron_MXH_MetalRings:MX100H
- SW65: value CPG151101S11 -> B; footprint acheron_MXH:MX225H -> acheron_MXH_MetalRings:MX100H
- SW66: value CPG151101S11 -> N; footprint acheron_MXH:MX100H -> acheron_MXH_MetalRings:MX100H
- SW67: value CPG151101S11 -> M; footprint acheron_MXH:MX100H -> acheron_MXH_MetalRings:MX100H
- SW68: value CPG151101S11 -> COMMA; footprint acheron_MXH:MX100H -> acheron_MXH_MetalRings:MX100H
- SW69: value CPG151101S11 -> DOT; footprint acheron_MXH:MX100H -> acheron_MXH_MetalRings:MX100H
- SW7: value CPG151101S11 -> F5; footprint acheron_MXH:MX100H -> acheron_MXH_MetalRings:MX100H
- SW70: value CPG151101S11 -> SLSH; footprint acheron_MXH:MX100H -> acheron_MXH_MetalRings:MX100H
- SW71: value CPG151101S11 -> RSHFT; footprint acheron_MXH:MX100H -> acheron_MXH_MetalRings:MX175H
- SW72: value CPG151101S11 -> UP; footprint acheron_MXH:MX100H -> acheron_MXH_MetalRings:MX100H
- SW73: value CPG151101S11 -> PGDN; footprint acheron_MXH:MX100H -> acheron_MXH_MetalRings:MX100H
- SW74: value CPG151101S11 -> LCTRL; footprint acheron_MXH:MX100H -> acheron_MXH_MetalRings:MX125H
- SW75: value CPG151101S11 -> WIN; footprint acheron_MXH:MX100H -> acheron_MXH_MetalRings:MX125H
- SW76: value CPG151101S11 -> LALT; footprint acheron_MXH:MX275H -> acheron_MXH_MetalRings:MX125H
- SW77: value CPG151101S11 -> SPACE; footprint acheron_MXH:MX100H -> acheron_MXH_MetalRings:MX625HR
- SW78: value CPG151101S11 -> RALT; footprint acheron_MXH:MX125H -> acheron_MXH_MetalRings:MX100H
- SW79: value CPG151101S11 -> FN; footprint acheron_MXH:MX125H -> acheron_MXH_MetalRings:MX100H
- SW8: value CPG151101S11 -> F6; footprint acheron_MXH:MX100H -> acheron_MXH_MetalRings:MX100H
- SW80: value CPG151101S11 -> RCTRL; footprint acheron_MXH:MX125H -> acheron_MXH_MetalRings:MX100H
- SW81: value CPG151101S11 -> LEFT; footprint acheron_MXH:MX625HR -> acheron_MXH_MetalRings:MX100H
- SW82: value CPG151101S11 -> DOWN; footprint acheron_MXH:MX125H -> acheron_MXH_MetalRings:MX100H
- SW83: value CPG151101S11 -> RIGHT; footprint acheron_MXH:MX125H -> acheron_MXH_MetalRings:MX100H
- SW9: value CPG151101S11 -> F7; footprint acheron_MXH:MX100H -> acheron_MXH_MetalRings:MX100H
- X5: footprint acheron_Connectors:PinHeader_1x3_P2.54mm_Vertical -> acheron_Connectors:PinHeader_1x3_staggered_P2.54mm_Vertical
Connections:
- net +3V3 is gone; now on net 3V3: J4.3 (VCC)
Other:
- company: Designed by Gondolindrim -> Designed by Hieu TN
- title: Apollo87H PCB schematic -> LONE PCB schematic

Commit message: place components
Parts:
- removed D16: 1N4148W, acheron_Components:D_SOD-123, symbol Device:D
- removed SW15: KNOB, acheron_MXH_MetalRings:MX100H, symbol acheronSymbols:Mechanical_Switch
- removed X4: EXTRA_PINS, acheron_Connectors:PinHeader_2x3_P2.54mm_Vertical_Staggered, symbol Connector_Generic:Conn_02x03_Odd_Even
Connections:
- no-connect marks 7 -> 4
Changed lines of the file:
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@@
   (junction (at 248.92 287.02) (diameter 1.016) (color 0 0 0 0)
   )
-  (junction (at 363.22 185.42) (diameter 1.016) (color 0 0 0 0)
-  )
   (junction (at 147.32 210.82) (diameter 1.016) (color 0 0 0 0)
   )
@@
   (junction (at 789.94 516.255) (diameter 0) (color 0 0 0 0)
   )
-  (junction (at 401.32 210.82) (diameter 1.016) (color 0 0 0 0)
-  )
   (junction (at 789.94 569.595) (diameter 0) (color 0 0 0 0)
   )
@@
   )
   (no_connect (at 185.42 101.6))
-  (no_connect (at 882.65 390.525))
   (no_connect (at 873.76 86.36))
   (no_connect (at 873.76 90.17))
-  (no_connect (at 895.35 387.985))
-  (no_connect (at 895.35 390.525))
   (no_connect (at 185.42 104.14))
   (wire (pts (xy 58.42 393.7) (xy 58.42 397.51))
@@
     (stroke (width 0) (type default) (color 0 0 0 0))
   )
-  (wire (pts (xy 401.32 172.72) (xy 401.32 210.82))
+  (wire (pts (xy 401.32 172.72) (xy 401.32 248.92))
     (stroke (width 0) (type solid) (color 0 0 0 0))
   )
@@
     (stroke (width 0) (type solid) (color 0 0 0 0))
   )
-  (wire (pts (xy 414.02 198.12) (xy 414.02 201.93))
-    (stroke (width 0) (type solid) (color 0 0 0 0))
-  )
   (wire (pts (xy 345.44 639.445) (xy 345.44 641.985))
     (stroke (width 0) (type default) (color 0 0 0 0))
@@
     (stroke (width 0) (type solid) (color 0 0 0 0))
   )
-  (wire (pts (xy 401.32 210.82) (xy 405.13 210.82))
-    (stroke (width 0) (type solid) (color 0 0 0 0))
-  )
   (wire (pts (xy 312.42 185.42) (xy 312.42 190.5))
     (stroke (width 0) (type solid) (color 0 0 0 0))
@@
     (stroke (width 0) (type solid) (color 0 0 0 0))
   )
-  (wire (pts (xy 401.32 210.82) (xy 401.32 248.92))
-    (stroke (width 0) (type solid) (color 0 0 0 0))
-  )
   (wire (pts (xy 401.32 248.92) (xy 401.32 287.02))
     (stroke (width 0) (type solid) (color 0 0 0 0))
@@
     (stroke (width 0) (type default) (color 0 0 0 0))
   )
-  (wire (pts (xy 363.22 185.42) (xy 414.02 185.42))
-    (stroke (width 0) (type solid) (color 0 0 0 0))
-  )
   (wire (pts (xy 96.52 123.825) (xy 96.52 127))
     (stroke (width 0) (type solid) (color 0 0 0 0))
@@
     (stroke (width 0) (type default) (color 0 0 0 0))
   )
-  (wire (pts (xy 414.02 185.42) (xy 414.02 190.5))
-    (stroke (width 0) (type solid) (color 0 0 0 0))
-  )
   (wire (pts (xy 388.62 393.7) (xy 388.62 397.51))
     (stroke (width 0) (type solid) (color 0 0 0 0))
@@
     )
   )
-  (global_label "E_PB13" (shape bidirectional) (at 882.65 393.065 180)
-    (effects (font (size 0.762 0.762)) (justify right))
-    (property "Intersheet References" "${INTERSHEET_REFS}" (id 0) (at 877.7574 393.1444 0)
-      (effects (font (size 0.762 0.762)) (justify right) hide)
-    )
-  )
   (global_label "E_PA14" (shape bidirectional) (at 782.32 279.4 90)
     (effects (font (size 1.27 1.27)) (justify left))
@@
     )
   )
-  (global_label "3V3" (shape input) (at 895.35 393.065 0)
-    (effects (font (size 0.762 0.762)) (justify left))
-    (property "Intersheet References" "${INTERSHEET_REFS}" (id 0) (at 898.9025 393.0174 0)
-      (effects (font (size 0.762 0.762)) (justify left) hide)
-    )
-  )
   (global_label "5V" (shape input) (at 567.69 610.87 90)
     (effects (font (size 1.27 1.27)) (justify left))
@@
     (pin "4")
   )
-  (symbol (lib_id "acheronSymbols:Mechanical_Switch") (at 414.02 210.82 0) (unit 1)
-    (in_bom yes) (on_board yes)
-    (property "Reference" "SW15" (id 0) (at 414.02 210.312 0))
-    (property "Value" "KNOB" (id 1) (at 414.02 214.63 0)
-      (effects (font (size 0.762 0.762)) hide)
-    )
-    (property "Footprint" "acheron_MXH_MetalRings:MX100H" (id 2) (at 414.02 210.82 0)
-      (effects (font (size 1.27 1.27)) hide)
-    )
-    (property "Datasheet" "" (id 3) (at 414.02 210.82 0)
-      (effects (font (size 1.27 1.27)) hide)
-    )
-    (property "Keycode" "KNOB" (id 7) (at 414.02 212.09 0)
-      (effects (font (size 0.762 0.762)))
-    )
-    (property "Manufacturer" "Kaihua" (id 8) (at 414.02 210.82 0)
-      (effects (font (size 1.27 1.27)) hide)
-    )
-    (property "Specification" "MX-style switch solderless (\"hotswap\") socket" (id 9) (at 414.02 210.82 0)
-      (effects (font (size 1.27 1.27)) hide)
-    )
-    (property "Manufacturer Part Number" "CPG151101S11" (id 10) (at 414.02 210.82 0)
-      (effects (font (size 1.27 1.27)) hide)
-    )
-    (pin "1")
-    (pin "2")
-  )
   (symbol (lib_id "acheron_Symbols:SK6812MINI-E") (at 656.59 578.485 0) (unit 1)
     (in_bom yes) (on_board yes)
@@
     (pin "1")
   )
-  (symbol (lib_id "Device:D") (at 414.02 194.31 270) (unit 1)
-    (in_bom yes) (on_board yes)
-    (property "Reference" "D16" (id 0) (at 419.5002 194.31 0))
-    (property "Value" "1N4148W" (id 1) (at 417.2015 194.31 0))
-    (property "Footprint" "acheron_Components:D_SOD-123" (id 2) (at 414.02 194.31 0)
-      (effects (font (size 1.27 1.27)) hide)
-    )
-    (property "Datasheet" "~" (id 3) (at 414.02 194.31 0)
-      (effects (font (size 1.27 1.27)) hide)
-    )
-    (property "Package" "SOD-123" (id 4) (at 414.02 194.31 0)
-      (effects (font (size 1.27 1.27)) hide)
-    )
-    (property "Specification" "Small-signal switching diodes" (id 5) (at 414.02 194.31 0)
-      (effects (font (size 1.27 1.27)) hide)
-    )
-    (pin "1")
-    (pin "2")
-  )
   (symbol (lib_id "power:GND") (at 624.205 569.595 90) (unit 1)
     (in_bom yes) (on_board yes)
@@
     (pin "1")
   )
-  (symbol (lib_id "power:GND") (at 882.65 387.985 270) (unit 1)
-    (in_bom yes) (on_board yes)
-    (property "Reference" "#PWR043" (id 0) (at 876.3 387.985 0)
-      (effects (font (size 1.27 1.27)) hide)
-    )
-    (property "Value" "GND" (id 1) (at 878.205 387.985 90)
-      (effects (font (size 0.762 0.762)))
-    )
-    (property "Footprint" "" (id 2) (at 882.65 387.985 0)
-      (effects (font (size 1.27 1.27)) hide)
-    )
-    (property "Datasheet" "" (id 3) (at 882.65 387.985 0)
-      (effects (font (size 1.27 1.27)) hide)
-    )
-    (pin "1")
-  )
   (symbol (lib_id "Device:R_Small") (at 834.39 615.315 180) (unit 1)
     (in_bom yes) (on_board yes)
@@
     (pin "2")
   )
-  (symbol (lib_id "Connector_Generic:Conn_02x03_Odd_Even") (at 887.73 390.525 0) (mirror x) (unit 1)
-    (in_bom no) (on_board yes)
-    (property "Reference" "X4" (id 0) (at 889 382.27 0))
-    (property "Value" "EXTRA_PINS" (id 1) (at 889 384.81 0))
-    (property "Footprint" "acheron_Connectors:PinHeader_2x3_P2.54mm_Vertical_Staggered" (id 2) (at 887.73 390.525 0)
-      (effects (font (size 1.27 1.27)) hide)
-    )
-    (property "Datasheet" "~" (id 3) (at 887.73 390.525 0)
-      (effects (font (size 1.27 1.27)) hide)
-    )
-    (property "LCSC Part Number" "" (id 6) (at 887.73 390.525 0)
-      (effects (font (size 1.27 1.27)) hide)
-    )
-    (property "Specification" "" (id 7) (at 887.73 390.525 0)
-      (effects (font (size 1.27 1.27)) hide)
-    )
-    (pin "1")
-    (pin "2")
-    (pin "3")
-    (pin "4")
-    (pin "5")
-    (pin "6")
-  )
   (symbol (lib_id "acheron_Symbols:SK6812MINI-E") (at 434.34 738.505 0) (mirror y) (unit 1)
     (in_bom yes) (on_board yes)
@@
       (reference "#PWR042") (unit 1) (value "GND") (footprint "")
     )
-    (path "/a440ce68-005d-4047-9fc4-322fbc5f560b"
-      (reference "#PWR043") (unit 1) (value "GND") (footprint "")
-    )
     (path "/89cb28de-ee0b-455c-b49b-c539400487fa"
       (reference "#PWR044") (unit 1) (value "GND") (footprint "")
@@
       (reference "D15") (unit 1) (value "1N4148W") (footprint "acheron_Components:D_SOD-123")
     )
-    (path "/78c7ca31-120f-4b6a-a11f-fb6e2bf2d9ea"
-      (reference "D16") (unit 1) (value "1N4148W") (footprint "acheron_Components:D_SOD-123")
-    )
     (path "/fef0f05f-600a-4ce4-9d3d-37e61e2ad45d"
       (reference "D17") (unit 1) (value "1N4148W") (footprint "acheron_Components:D_SOD-123")
@@
       (reference "SW14") (unit 1) (value "F12") (footprint "acheron_MXH_MetalRings:MX100H")
     )
-    (path "/6f0e1a7e-e2ec-483b-9f29-66f7a43483ef"
-      (reference "SW15") (unit 1) (value "KNOB") (footprint "acheron_MXH_MetalRings:MX100H")
-    )
     (path "/551c55ec-026e-44c3-9f46-bf7b41fc5f08"
       (reference "SW16") (unit 1) (value "GRV") (footprint "acheron_MXH_MetalRings:MX100H")
@@
       (reference "X3") (unit 1) (value "EXTRA_PINS") (footprint "acheron_Connectors:PinHeader_1x16_P2.54mm_Vertical")
     )
-    (path "/db969484-34e6-4e3f-b6d7-af072dc78e5c"
-      (reference "X4") (unit 1) (value "EXTRA_PINS") (footprint "acheron_Connectors:PinHeader_2x3_P2.54mm_Vertical_Staggered")
-    )
     (path "/a8de232c-c704-422f-a90e-f3b71b8d496b"

Commit message: routing
Parts:
- added D16: 1N4148W, acheron_Components:D_SOD-123, symbol Device:D
- added SW15: KNOB, acheron_MXA:MXA100, symbol acheronSymbols:Mechanical_Switch
Connections:
- net C0: now also U4.33 (PB12); no longer U4.39 (USART6_CK/TIM3_CH3/PC8)
- net C1: now also U4.35 (SPI2_MISO/PB14); no longer U4.40 (TIM3_CH4/I2S_CKIN/PC9)
- net C10: now also U4.10 (PC2/SPI2_MISO); no longer U4.25 (PC5)
- net C11: now also U4.11 (PC3/SPI2_MOSI); no longer U4.24 (PC4)
- net C12: now also U4.14 (PA0/TIM2_CH1/USART2_CTS); no longer U4.23 (PA7/SPI1_MOSI/TIM3_CH2)
- net C13: now also U4.15 (PA1/TIM2_CH2/USART2_RTS); no longer U4.26 (PB0/TIM3_CH3)
- net C14: now also U4.16 (PA2/TIM2_CH3/USART2_TX), SW15.1; no longer U4.52 (SPI3_MISO/PC11)
- net C2: now also U4.37 (I2S2_MCK/TIM3_CH1/USART6_TX/PC6); no longer U4.41 (USART1_CK/TIM1_CH1/PA8)
- net C3: now also U4.38 (USART6_RX/TIM3_CH2/PC7); no longer U4.43 (USART1_RX/TIM1_CH3/PA10)
- net C4: now also U4.39 (USART6_CK/TIM3_CH3/PC8); no longer U4.38 (USART6_RX/TIM3_CH2/PC7)
- net C5: now also U4.40 (TIM3_CH4/I2S_CKIN/PC9); no longer U4.37 (I2S2_MCK/TIM3_CH1/USART6_TX/PC6)
- net C6: now also U4.41 (USART1_CK/TIM1_CH1/PA8); no longer U4.35 (SPI2_MISO/PB14)
- net C7: now also U4.43 (USART1_RX/TIM1_CH3/PA10); no longer U4.33 (PB12)
- net C8: now also U4.8 (PC0); no longer U4.29 (PB10/TIM2_CH3/SPI2_SCK/I2C2_SCL/I2S2_CK)
- net C9: now also U4.9 (PC1); no longer U4.27 (PB1/TIM3_CH4)
- net E_PA14: no longer U4.50 (JTDI/TIM2_CH1/PA14)
- net E_PA3: now also X3.5 (Pin_5); no longer X3.13 (Pin_13)
- net PA9: no longer X3.14 (Pin_14)
- net R0: now also D16.1 (K)
- net R3: now also U4.52 (SPI3_MISO/PC11); no longer U4.22 (PA6/TIM3_CH1/SPI1_MISO)
- net R4: now also U4.51 (SPI3_SCK/I2S3_CK/PC10); no longer U4.21 (PA5/TIM2_CH1/SPI1_SCK)
- net R5: now also U4.50 (JTDI/TIM2_CH1/PA14); no longer U4.20 (PA4/USART2_CK)
- net E_PA0 renamed E_PC4
- net E_PC4: now also U4.24 (PC4); no longer U4.14 (PA0/TIM2_CH1/USART2_CTS)
- net E_PA1 renamed E_PC5
- net E_PC5: now also U4.25 (PC5); no longer U4.15 (PA1/TIM2_CH2/USART2_RTS)
- net E_PA2 renamed E_PB0
- net E_PB0: now also U4.26 (PB0/TIM3_CH3); no longer U4.16 (PA2/TIM2_CH3/USART2_TX)
- removed net E_PC0: U4.8 (PC0), X3.5 (Pin_5)
- net E_PC1 renamed E_PA4
- net E_PA4: now also U4.20 (PA4/USART2_CK); no longer U4.9 (PC1)
- net E_PC10 renamed E_PA7
- net E_PA7: now also U4.23 (PA7/SPI1_MOSI/TIM3_CH2); no longer U4.51 (SPI3_SCK/I2S3_CK/PC10)
- net E_PC2 renamed E_PA5
- net E_PA5: now also U4.21 (PA5/TIM2_CH1/SPI1_SCK); no longer U4.10 (PC2/SPI2_MISO)
- net E_PC3 renamed E_PA6
- net E_PA6: now also U4.22 (PA6/TIM3_CH1/SPI1_MISO); no longer U4.11 (PC3/SPI2_MOSI)
- new net: D16.2 (A), SW15.2
- new net E_PB1: U4.27 (PB1/TIM3_CH4), X3.13 (Pin_13)
- new net E_PB10: U4.29 (PB10/TIM2_CH3/SPI2_SCK/I2C2_SCL/I2S2_CK), X3.14 (Pin_14)
