File: kb-lone.kicad_sch (KiCad schematic)
At the start: 474 parts, among them J1 TYPE-C-31-M12, J2 SM04B-SRSS-TB(LF)(SN), J3 SM04B-SRSS-TB(LF)(SN), J4 SSD1306, M1 RGB DB notch, Q1 DTC123JKAT146, SW1 K2-1187SQ-A4SW-06, SW10 F8, SW11 F9, SW12 F10, SW13 F11, SW14 F12, SW15 KNOB, SW16 GRV, SW17 1, SW18 2, SW19 3, SW2 ESC, SW20 4, SW21 5, SW22 6, SW23 7, SW24 8, SW25 9, SW26 0, SW27 MINUS, SW28 EQUAL, SW29 BSPC, SW3 F1, SW30 N/A, SW31 TAB, SW32 Q, SW33 W, SW34 E, SW35 R, SW36 T, SW37 Y, SW38 U, SW39 I, SW4 F2, SW40 O, SW41 P, SW42 LBRKT, SW43 RBRKT, SW44 BSLS, SW45 N/A, SW46 CAPS, SW47 A, SW48 S, SW49 D, SW5 F3, SW50 F, SW51 G, SW52 H, SW53 J, SW54 K, SW55 L, SW56 COLON, SW57 QUOTE, SW58 ENTER, SW59 PGUP, SW6 F4, SW60 LSHFT, SW61 Z, SW62 X, SW63 C, SW64 V, SW65 B, SW66 N, SW67 M, SW68 COMMA, SW69 DOT, SW7 F5, SW70 SLSH, SW71 RSHFT, SW72 UP, SW73 PGDN, SW74 LCTRL, SW75 WIN, SW76 LALT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

Commit message: routing
Parts:
- removed X2: ARM JTAG, acheron_Connectors:PinHeader_2x5_P2.54mm_Vertical_Staggered, symbol Connector_Generic:Conn_02x05_Odd_Even
- removed X3: EXTRA_PINS, acheron_Connectors:PinHeader_1x16_P2.54mm_Vertical, symbol Connector_Generic:Conn_01x16
- removed X5: Conn_01x03, acheron_Connectors:PinHeader_1x3_staggered_P2.54mm_Vertical, symbol Connector_Generic:Conn_01x03
Connections:
- net E_PB4 is gone; now on net R1: U4.56 (NJTRST/SPI1_MISO/SPI3_MISO/I2C3_SDA/TIM3_CH1/PB4)
- net SWCLK is gone; now on net ENC_SW: U4.49 (JTCK-SWCLK/PA14)
- net ENC_A: now also U4.51 (SPI3_SCK/I2S3_CK/PC10); no longer U4.57 (SPI1_MOSI/SPI3_MOSI/TIM3_CH2/PB5)
- net ENC_B: now also U4.50 (JTDI/TIM2_CH1/PA14); no longer U4.61 (I2C1_SCL/TIM4_CH3/TIM10_CH1/PB8)
- net ENC_SW: no longer U4.62 (I2C1_SDA/TIM4_CH4/TIM11_CH1/PB9)
- net R0: now also U4.57 (SPI1_MOSI/SPI3_MOSI/TIM3_CH2/PB5); no longer U4.55 (JTDO-SWO/SPI1_SCK/SPI3_SCK/I2C2_SDA/TIM2_CH2/PB3)
- net R1: no longer U4.54 (PD2)
- net R2: now also U4.55 (JTDO-SWO/SPI1_SCK/SPI3_SCK/I2C2_SDA/TIM2_CH2/PB3); no longer U4.53 (SPI3_MOSI/PC12)
- net R3: now also U4.54 (PD2); no longer U4.52 (SPI3_MISO/PC11)
- net R4: now also U4.53 (SPI3_MOSI/PC12); no longer U4.51 (SPI3_SCK/I2S3_CK/PC10)
- net R5: now also U4.52 (SPI3_MISO/PC11); no longer U4.50 (JTDI/TIM2_CH1/PA14)
- net at D128.2 (DOUT): now also D127.4 (DIN); no longer D113.2 (DOUT)
- net at D128.4 (DIN): now also D113.2 (DOUT); no longer D127.2 (DOUT)
- net at D158.2 (DOUT): now also D159.4 (DIN); no longer D157.4 (DIN)
- net at D158.4 (DIN): now also D157.2 (DOUT); no longer D159.2 (DOUT)
- net at D138.2 (DOUT): now also D139.4 (DIN); no longer D137.2 (DOUT)
- net at D138.4 (DIN): now also D137.2 (DOUT); no longer D139.2 (DOUT)
- net at D126.2 (DOUT): now also D125.4 (DIN); no longer D127.4 (DIN)
- net at D126.4 (DIN): now also D127.2 (DOUT); no longer D125.2 (DOUT)
- net at D143.2 (DOUT): now also D157.4 (DIN); no longer D157.2 (DOUT)
- net at D141.2 (DOUT): now also D142.4 (DIN); no longer D140.4 (DIN)
- net at D141.4 (DIN): now also D140.2 (DOUT); no longer D142.2 (DOUT)
- net at D156.2 (DOUT): now also D155.4 (DIN); no longer D142.4 (DIN)
- net at D99.2 (DOUT): now also D100.4 (DIN); no longer D85.2 (DOUT)
- net at D99.4 (DIN): now also D85.2 (DOUT); no longer D100.2 (DOUT)
- net at D160.4 (DIN): now also D159.2 (DOUT); no longer D159.4 (DIN)
- net at D156.4 (DIN): now also D142.2 (DOUT); no longer D155.2 (DOUT)
- net at D154.2 (DOUT): now also D153.4 (DIN); no longer D155.4 (DIN)
- net at D124.4 (DIN): now also D125.2 (DOUT); no longer D125.4 (DIN)
- net at D154.4 (DIN): now also D155.2 (DOUT); no longer D153.2 (DOUT)
- net at D152.4 (DIN): now also D153.2 (DOUT); no longer D153.4 (DIN)
- net at D101.4 (DIN): now also D100.2 (DOUT); no longer D100.4 (DIN)
- new net: D139.2 (DOUT), D140.4 (DIN)
- new net E_PB8: U4.61 (I2C1_SCL/TIM4_CH3/TIM10_CH1/PB8)
- new net E_PB9: U4.62 (I2C1_SDA/TIM4_CH4/TIM11_CH1/PB9)

Commit message: routing
Connections:
- net E_PB8 is gone; now on net RGB_3V3: U4.61 (I2C1_SCL/TIM4_CH3/TIM10_CH1/PB8)
- net C0: now also U4.35 (SPI2_MISO/PB14); no longer U4.33 (PB12)
- net C1: now also U4.36 (SPI2_MOSI/PB15); no longer U4.35 (SPI2_MISO/PB14)
- net RGB_3V3: no longer U4.36 (SPI2_MOSI/PB15)
- new net E_PB12: U4.33 (PB12)
Changed lines of the file:
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@@
     )
   )
-  (global_label "E_PB8" (shape bidirectional) (at 712.47 279.4 90) (fields_autoplaced)
-    (effects (font (size 1.27 1.27)) (justify left))
-    (property "Intersheet References" "${INTERSHEET_REFS}" (id 0) (at 712.3906 271.1207 90)
+  (global_label "E_PB9" (shape bidirectional) (at 706.12 279.4 90) (fields_autoplaced)
+    (effects (font (size 1.27 1.27)) (justify left))
+    (property "Intersheet References" "${INTERSHEET_REFS}" (id 0) (at 706.0406 271.1207 90)
       (effects (font (size 1.27 1.27)) (justify left) hide)
     )
@@
     )
   )
-  (global_label "C0" (shape output) (at 797.56 383.54 0)
+  (global_label "C0" (shape output) (at 797.56 370.84 0)
     (effects (font (size 1.524 1.524)) (justify left))
-    (property "Intersheet References" "${INTERSHEET_REFS}" (id 0) (at 815.5155 383.4606 0)
+    (property "Intersheet References" "${INTERSHEET_REFS}" (id 0) (at 815.5155 370.7606 0)
       (effects (font (size 1.524 1.524)) (justify left) hide)
     )
@@
     )
   )
-  (global_label "RGB_3V3" (shape output) (at 797.56 364.49 0)
-    (effects (font (size 1.27 1.27)) (justify left))
-    (property "Intersheet References" "${INTERSHEET_REFS}" (id 0) (at 856.615 751.84 0)
-      (effects (font (size 1.27 1.27)) hide)
+  (global_label "RGB_3V3" (shape output) (at 712.47 279.4 90)
+    (effects (font (size 1.27 1.27)) (justify left))
+    (property "Intersheet References" "${INTERSHEET_REFS}" (id 0) (at 325.12 220.345 90)
+      (effects (font (size 1.27 1.27)) (justify right) hide)
     )
   )
@@
     )
   )
-  (global_label "E_PB9" (shape bidirectional) (at 706.12 279.4 90)
-    (effects (font (size 1.27 1.27)) (justify left))
-    (property "Intersheet References" "${INTERSHEET_REFS}" (id 0) (at 706.0406 270.7579 90)
+  (global_label "E_PB13" (shape bidirectional) (at 797.56 377.19 0)
+    (effects (font (size 1.27 1.27)) (justify left))
+    (property "Intersheet References" "${INTERSHEET_REFS}" (id 0) (at 806.2021 377.1106 0)
       (effects (font (size 1.27 1.27)) (justify left) hide)
     )
@@
     )
   )
-  (global_label "E_PB13" (shape bidirectional) (at 797.56 377.19 0)
-    (effects (font (size 1.27 1.27)) (justify left))
-    (property "Intersheet References" "${INTERSHEET_REFS}" (id 0) (at 802.4526 377.1106 0)
+  (global_label "E_PB12" (shape bidirectional) (at 797.56 383.54 0)
+    (effects (font (size 1.27 1.27)) (justify left))
+    (property "Intersheet References" "${INTERSHEET_REFS}" (id 0) (at 802.4526 383.4606 0)
       (effects (font (size 1.27 1.27)) (justify left) hide)
     )
@@
     )
   )
-  (global_label "C1" (shape output) (at 797.56 370.84 0)
+  (global_label "C1" (shape output) (at 797.56 364.49 0)
     (effects (font (size 1.524 1.524)) (justify left))
-    (property "Intersheet References" "${INTERSHEET_REFS}" (id 0) (at 815.5155 370.7606 0)
+    (property "Intersheet References" "${INTERSHEET_REFS}" (id 0) (at 815.5155 364.4106 0)
       (effects (font (size 1.524 1.524)) (justify left) hide)
     )

Commit message: routing
Connections:
- net C10: now also U4.54 (PD2); no longer U4.10 (PC2/SPI2_MISO)
- net C11: now also U4.55 (JTDO-SWO/SPI1_SCK/SPI3_SCK/I2C2_SDA/TIM2_CH2/PB3); no longer U4.11 (PC3/SPI2_MOSI)
- net C12: now also U4.56 (NJTRST/SPI1_MISO/SPI3_MISO/I2C3_SDA/TIM3_CH1/PB4); no longer U4.14 (PA0/TIM2_CH1/USART2_CTS)
- net C13: now also U4.57 (SPI1_MOSI/SPI3_MOSI/TIM3_CH2/PB5); no longer U4.15 (PA1/TIM2_CH2/USART2_RTS)
- net C8: now also U4.52 (SPI3_MISO/PC11); no longer U4.8 (PC0)
- net C9: now also U4.53 (SPI3_MOSI/PC12); no longer U4.9 (PC1)
- net R0: now also U4.8 (PC0); no longer U4.57 (SPI1_MOSI/SPI3_MOSI/TIM3_CH2/PB5)
- net R1: now also U4.9 (PC1); no longer U4.56 (NJTRST/SPI1_MISO/SPI3_MISO/I2C3_SDA/TIM3_CH1/PB4)
- net R2: now also U4.10 (PC2/SPI2_MISO); no longer U4.55 (JTDO-SWO/SPI1_SCK/SPI3_SCK/I2C2_SDA/TIM2_CH2/PB3)
- net R3: now also U4.11 (PC3/SPI2_MOSI); no longer U4.54 (PD2)
- net R4: now also U4.14 (PA0/TIM2_CH1/USART2_CTS); no longer U4.53 (SPI3_MOSI/PC12)
- net R5: now also U4.15 (PA1/TIM2_CH2/USART2_RTS); no longer U4.52 (SPI3_MISO/PC11)
Changed lines of the file:
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@@
     )
   )
-  (global_label "R2" (shape input) (at 750.57 279.4 90)
-    (effects (font (size 1.27 1.27)) (justify left))
-    (property "Intersheet References" "${INTERSHEET_REFS}" (id 0) (at 750.4906 274.5074 90)
-      (effects (font (size 1.27 1.27)) (justify left) hide)
+  (global_label "R2" (shape input) (at 684.53 345.44 180)
+    (effects (font (size 1.27 1.27)) (justify right))
+    (property "Intersheet References" "${INTERSHEET_REFS}" (id 0) (at 679.6374 345.5194 0)
+      (effects (font (size 1.27 1.27)) (justify right) hide)
     )
   )
@@
     )
   )
-  (global_label "R3" (shape input) (at 756.92 279.4 90)
-    (effects (font (size 1.27 1.27)) (justify left))
-    (property "Intersheet References" "${INTERSHEET_REFS}" (id 0) (at 756.9994 274.5074 90)
-      (effects (font (size 1.27 1.27)) (justify left) hide)
+  (global_label "R3" (shape input) (at 684.53 351.79 180)
+    (effects (font (size 1.27 1.27)) (justify right))
+    (property "Intersheet References" "${INTERSHEET_REFS}" (id 0) (at 679.6374 351.7106 0)
+      (effects (font (size 1.27 1.27)) (justify right) hide)
     )
   )
@@
     )
   )
-  (global_label "C12" (shape output) (at 684.53 370.84 180)
-    (effects (font (size 1.27 1.27)) (justify right))
-    (property "Intersheet References" "${INTERSHEET_REFS}" (id 0) (at 679.6374 370.9194 0)
-      (effects (font (size 1.27 1.27)) (justify right) hide)
+  (global_label "C12" (shape output) (at 744.22 279.4 90)
+    (effects (font (size 1.27 1.27)) (justify left))
+    (property "Intersheet References" "${INTERSHEET_REFS}" (id 0) (at 744.1406 274.5074 90)
+      (effects (font (size 1.27 1.27)) (justify left) hide)
     )
   )
@@
     )
   )
-  (global_label "R5" (shape input) (at 769.62 279.4 90)
-    (effects (font (size 1.27 1.27)) (justify left))
-    (property "Intersheet References" "${INTERSHEET_REFS}" (id 0) (at 769.5406 274.5074 90)
-      (effects (font (size 1.27 1.27)) (justify left) hide)
+  (global_label "R5" (shape input) (at 684.53 377.19 180)
+    (effects (font (size 1.27 1.27)) (justify right))
+    (property "Intersheet References" "${INTERSHEET_REFS}" (id 0) (at 679.6374 377.2694 0)
+      (effects (font (size 1.27 1.27)) (justify right) hide)
     )
   )
@@
     )
   )
-  (global_label "C8" (shape output) (at 684.53 332.74 180)
-    (effects (font (size 1.27 1.27)) (justify right))
-    (property "Intersheet References" "${INTERSHEET_REFS}" (id 0) (at 679.6374 332.8194 0)
-      (effects (font (size 1.27 1.27)) (justify right) hide)
+  (global_label "C8" (shape output) (at 769.62 279.4 90)
+    (effects (font (size 1.27 1.27)) (justify left))
+    (property "Intersheet References" "${INTERSHEET_REFS}" (id 0) (at 769.5406 274.5074 90)
+      (effects (font (size 1.27 1.27)) (justify left) hide)
     )
   )
@@
     )
   )
-  (global_label "C10" (shape output) (at 684.53 345.44 180)
-    (effects (font (size 1.27 1.27)) (justify right))
-    (property "Intersheet References" "${INTERSHEET_REFS}" (id 0) (at 679.6374 345.5194 0)
-      (effects (font (size 1.27 1.27)) (justify right) hide)
+  (global_label "C10" (shape output) (at 756.92 279.4 90)
+    (effects (font (size 1.27 1.27)) (justify left))
+    (property "Intersheet References" "${INTERSHEET_REFS}" (id 0) (at 756.8406 274.5074 90)
+      (effects (font (size 1.27 1.27)) (justify left) hide)
     )
   )
@@
     )
   )
-  (global_label "C9" (shape output) (at 684.53 339.09 180)
-    (effects (font (size 1.27 1.27)) (justify right))
-    (property "Intersheet References" "${INTERSHEET_REFS}" (id 0) (at 679.6374 339.1694 0)
-      (effects (font (size 1.27 1.27)) (justify right) hide)
+  (global_label "C9" (shape output) (at 763.27 279.4 90)
+    (effects (font (size 1.27 1.27)) (justify left))
+    (property "Intersheet References" "${INTERSHEET_REFS}" (id 0) (at 763.1906 274.5074 90)
+      (effects (font (size 1.27 1.27)) (justify left) hide)
     )
   )
@@
     )
   )
-  (global_label "C13" (shape output) (at 684.53 377.19 180)
-    (effects (font (size 1.27 1.27)) (justify right))
-    (property "Intersheet References" "${INTERSHEET_REFS}" (id 0) (at 679.6374 377.2694 0)
-      (effects (font (size 1.27 1.27)) (justify right) hide)
+  (global_label "C13" (shape output) (at 737.87 279.4 90)
+    (effects (font (size 1.27 1.27)) (justify left))
+    (property "Intersheet References" "${INTERSHEET_REFS}" (id 0) (at 737.7906 274.5074 90)
+      (effects (font (size 1.27 1.27)) (justify left) hide)
     )
   )
@@
     )
   )
-  (global_label "C11" (shape output) (at 684.53 351.79 180)
-    (effects (font (size 1.27 1.27)) (justify right))
-    (property "Intersheet References" "${INTERSHEET_REFS}" (id 0) (at 679.6374 351.8694 0)
-      (effects (font (size 1.27 1.27)) (justify right) hide)
+  (global_label "C11" (shape output) (at 750.57 279.4 90)
+    (effects (font (size 1.27 1.27)) (justify left))
+    (property "Intersheet References" "${INTERSHEET_REFS}" (id 0) (at 750.4906 274.5074 90)
+      (effects (font (size 1.27 1.27)) (justify left) hide)
     )
   )
@@
     )
   )
-  (global_label "R1" (shape input) (at 744.22 279.4 90)
-    (effects (font (size 1.27 1.27)) (justify left))
-    (property "Intersheet References" "${INTERSHEET_REFS}" (id 0) (at 744.1406 274.5074 90)
-      (effects (font (size 1.27 1.27)) (justify left) hide)
+  (global_label "R1" (shape input) (at 684.53 339.09 180)
+    (effects (font (size 1.27 1.27)) (justify right))
+    (property "Intersheet References" "${INTERSHEET_REFS}" (id 0) (at 679.6374 339.1694 0)
+      (effects (font (size 1.27 1.27)) (justify right) hide)
     )
   )
@@
     )
   )
-  (global_label "R0" (shape input) (at 737.87 279.4 90)
-    (effects (font (size 1.27 1.27)) (justify left))
-    (property "Intersheet References" "${INTERSHEET_REFS}" (id 0) (at 737.7906 274.5074 90)
-      (effects (font (size 1.27 1.27)) (justify left) hide)
+  (global_label "R0" (shape input) (at 684.53 332.74 180)
+    (effects (font (size 1.27 1.27)) (justify right))
+    (property "Intersheet References" "${INTERSHEET_REFS}" (id 0) (at 679.6374 332.8194 0)
+      (effects (font (size 1.27 1.27)) (justify right) hide)
     )
   )
@@
     )
   )
-  (global_label "R4" (shape input) (at 763.27 279.4 90)
-    (effects (font (size 1.27 1.27)) (justify left))
-    (property "Intersheet References" "${INTERSHEET_REFS}" (id 0) (at 763.1906 274.5074 90)
-      (effects (font (size 1.27 1.27)) (justify left) hide)
-    )
-  )
+  (global_label "R4" (shape input) (at 684.53 370.84 180)
+    (effects (font (size 1.27 1.27)) (justify right))
+    (property "Intersheet References" "${INTERSHEET_REFS}" (id 0) (at 679.6374 370.9194 0)
+      (effects (font (size 1.27 1.27)) (justify right) hide)
+    )
+  )
