File: kb-lone.kicad_sch (KiCad schematic)
At the start: 471 parts, among them J1 TYPE-C-31-M12, J2 SM04B-SRSS-TB(LF)(SN), J3 SM04B-SRSS-TB(LF)(SN), J4 SSD1306, M1 RGB DB notch, Q1 DTC123JKAT146, SW1 K2-1187SQ-A4SW-06, SW10 F8, SW11 F9, SW12 F10, SW13 F11, SW14 F12, SW15 KNOB, SW16 GRV, SW17 1, SW18 2, SW19 3, SW2 ESC, SW20 4, SW21 5, SW22 6, SW23 7, SW24 8, SW25 9, SW26 0, SW27 MINUS, SW28 EQUAL, SW29 BSPC, SW3 F1, SW30 N/A, SW31 TAB, SW32 Q, SW33 W, SW34 E, SW35 R, SW36 T, SW37 Y, SW38 U, SW39 I, SW4 F2, SW40 O, SW41 P, SW42 LBRKT, SW43 RBRKT, SW44 BSLS, SW45 N/A, SW46 CAPS, SW47 A, SW48 S, SW49 D, SW5 F3, SW50 F, SW51 G, SW52 H, SW53 J, SW54 K, SW55 L, SW56 COLON, SW57 QUOTE, SW58 ENTER, SW59 PGUP, SW6 F4, SW60 LSHFT, SW61 Z, SW62 X, SW63 C, SW64 V, SW65 B, SW66 N, SW67 M, SW68 COMMA, SW69 DOT, SW7 F5, SW70 SLSH, SW71 RSHFT, SW72 UP, SW73 PGDN, SW74 LCTRL, SW75 WIN, SW76 LALT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

Commit message: routing
Parts:
- removed H2, H3, H4, H5, H6, H7, H8: 9774035243R, acheron_Hardware:9774035243R, symbol Mechanical:MountingHole
Changed lines of the file:
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@@
     (pin "1")
   )
-  (symbol (lib_id "Mechanical:MountingHole") (at 279.4 82.55 0) (unit 1)
-    (in_bom yes) (on_board yes)
-    (property "Reference" "H3" (id 0) (at 283.21 81.9149 0)
-      (effects (font (size 1.27 1.27)) (justify left))
-    )
-    (property "Value" "9774035243R" (id 1) (at 283.21 84.4549 0)
-      (effects (font (size 1.27 1.27)) (justify left))
-    )
-    (property "Footprint" "acheron_Hardware:9774035243R" (id 2) (at 279.4 82.55 0)
-      (effects (font (size 1.27 1.27)) hide)
-    )
-    (property "Datasheet" "~" (id 3) (at 279.4 82.55 0)
-      (effects (font (size 1.27 1.27)) hide)
-    )
-    (property "Manufacturer" "Wurth Elektronik" (id 4) (at 279.4 82.55 0)
-      (effects (font (size 1.27 1.27)) hide)
-    )
-    (property "Manufacturer Part Number" "9774030243R" (id 5) (at 279.4 82.55 0)
-      (effects (font (size 1.27 1.27)) hide)
-    )
-    (property "Specification" "3.5mm length M2 threaded surface mounted steel standoffs " (id 6) (at 279.4 82.55 0)
-      (effects (font (size 1.27 1.27)) hide)
-    )
-  )
   (symbol (lib_id "Device:R_Small") (at 478.79 561.975 180) (unit 1)
     (in_bom yes) (on_board yes)
@@
     (pin "2")
   )
-  (symbol (lib_id "Mechanical:MountingHole") (at 279.4 101.6 0) (unit 1)
-    (in_bom yes) (on_board yes)
-    (property "Reference" "H6" (id 0) (at 283.21 100.9649 0)
-      (effects (font (size 1.27 1.27)) (justify left))
-    )
-    (property "Value" "9774035243R" (id 1) (at 283.21 103.5049 0)
-      (effects (font (size 1.27 1.27)) (justify left))
-    )
-    (property "Footprint" "acheron_Hardware:9774035243R" (id 2) (at 279.4 101.6 0)
-      (effects (font (size 1.27 1.27)) hide)
-    )
-    (property "Datasheet" "~" (id 3) (at 279.4 101.6 0)
-      (effects (font (size 1.27 1.27)) hide)
-    )
-    (property "Manufacturer" "Wurth Elektronik" (id 4) (at 279.4 101.6 0)
-      (effects (font (size 1.27 1.27)) hide)
-    )
-    (property "Manufacturer Part Number" "9774030243R" (id 5) (at 279.4 101.6 0)
-      (effects (font (size 1.27 1.27)) hide)
-    )
-    (property "Specification" "3.5mm length M2 threaded surface mounted steel standoffs " (id 6) (at 279.4 101.6 0)
-      (effects (font (size 1.27 1.27)) hide)
-    )
-  )
   (symbol (lib_id "power:GND") (at 631.825 294.64 180) (unit 1)
     (in_bom yes) (on_board yes)
@@
     (pin "2")
   )
-  (symbol (lib_id "Mechanical:MountingHole") (at 279.4 76.2 0) (unit 1)
-    (in_bom yes) (on_board yes)
-    (property "Reference" "H2" (id 0) (at 283.21 75.5649 0)
-      (effects (font (size 1.27 1.27)) (justify left))
-    )
-    (property "Value" "9774035243R" (id 1) (at 283.21 78.1049 0)
-      (effects (font (size 1.27 1.27)) (justify left))
-    )
-    (property "Footprint" "acheron_Hardware:9774035243R" (id 2) (at 279.4 76.2 0)
-      (effects (font (size 1.27 1.27)) hide)
-    )
-    (property "Datasheet" "~" (id 3) (at 279.4 76.2 0)
-      (effects (font (size 1.27 1.27)) hide)
-    )
-    (property "Manufacturer" "Wurth Elektronik" (id 4) (at 279.4 76.2 0)
-      (effects (font (size 1.27 1.27)) hide)
-    )
-    (property "Manufacturer Part Number" "9774030243R" (id 5) (at 279.4 76.2 0)
-      (effects (font (size 1.27 1.27)) hide)
-    )
-    (property "Specification" "3.5mm length M2 threaded surface mounted steel standoffs " (id 6) (at 279.4 76.2 0)
-      (effects (font (size 1.27 1.27)) hide)
-    )
-  )
   (symbol (lib_id "power:GND") (at 523.24 535.305 0) (unit 1)
     (in_bom yes) (on_board yes)
@@
     (pin "1")
   )
-  (symbol (lib_id "Mechanical:MountingHole") (at 279.4 107.95 0) (unit 1)
-    (in_bom yes) (on_board yes)
-    (property "Reference" "H7" (id 0) (at 283.21 107.3149 0)
-      (effects (font (size 1.27 1.27)) (justify left))
-    )
-    (property "Value" "9774035243R" (id 1) (at 283.21 109.8549 0)
-      (effects (font (size 1.27 1.27)) (justify left))
-    )
-    (property "Footprint" "acheron_Hardware:9774035243R" (id 2) (at 279.4 107.95 0)
-      (effects (font (size 1.27 1.27)) hide)
-    )
-    (property "Datasheet" "~" (id 3) (at 279.4 107.95 0)
-      (effects (font (size 1.27 1.27)) hide)
-    )
-    (property "Manufacturer" "Wurth Elektronik" (id 4) (at 279.4 107.95 0)
-      (effects (font (size 1.27 1.27)) hide)
-    )
-    (property "Manufacturer Part Number" "9774030243R" (id 5) (at 279.4 107.95 0)
-      (effects (font (size 1.27 1.27)) hide)
-    )
-    (property "Specification" "3.5mm length M2 threaded surface mounted steel standoffs " (id 6) (at 279.4 107.95 0)
-      (effects (font (size 1.27 1.27)) hide)
-    )
-  )
   (symbol (lib_id "acheronSymbols:Mechanical_Switch") (at 363.22 287.02 0) (unit 1)
     (in_bom yes) (on_board yes)
@@
     (pin "2")
   )
-  (symbol (lib_id "Mechanical:MountingHole") (at 279.4 114.3 0) (unit 1)
-    (in_bom yes) (on_board yes)
-    (property "Reference" "H8" (id 0) (at 283.21 113.6649 0)
-      (effects (font (size 1.27 1.27)) (justify left))
-    )
-    (property "Value" "9774035243R" (id 1) (at 283.21 116.2049 0)
-      (effects (font (size 1.27 1.27)) (justify left))
-    )
-    (property "Footprint" "acheron_Hardware:9774035243R" (id 2) (at 279.4 114.3 0)
-      (effects (font (size 1.27 1.27)) hide)
-    )
-    (property "Datasheet" "~" (id 3) (at 279.4 114.3 0)
-      (effects (font (size 1.27 1.27)) hide)
-    )
-    (property "Manufacturer" "Wurth Elektronik" (id 4) (at 279.4 114.3 0)
-      (effects (font (size 1.27 1.27)) hide)
-    )
-    (property "Manufacturer Part Number" "9774030243R" (id 5) (at 279.4 114.3 0)
-      (effects (font (size 1.27 1.27)) hide)
-    )
-    (property "Specification" "3.5mm length M2 threaded surface mounted steel standoffs " (id 6) (at 279.4 114.3 0)
-      (effects (font (size 1.27 1.27)) hide)
-    )
-  )
   (symbol (lib_id "power:GND") (at 673.1 358.14 270) (unit 1)
     (in_bom yes) (on_board yes)
@@
     (pin "1")
   )
-  (symbol (lib_id "Mechanical:MountingHole") (at 279.4 95.25 0) (unit 1)
-    (in_bom yes) (on_board yes)
-    (property "Reference" "H5" (id 0) (at 283.21 94.6149 0)
-      (effects (font (size 1.27 1.27)) (justify left))
-    )
-    (property "Value" "9774035243R" (id 1) (at 283.21 97.1549 0)
-      (effects (font (size 1.27 1.27)) (justify left))
-    )
-    (property "Footprint" "acheron_Hardware:9774035243R" (id 2) (at 279.4 95.25 0)
-      (effects (font (size 1.27 1.27)) hide)
-    )
-    (property "Datasheet" "~" (id 3) (at 279.4 95.25 0)
-      (effects (font (size 1.27 1.27)) hide)
-    )
-    (property "Manufacturer" "Wurth Elektronik" (id 4) (at 279.4 95.25 0)
-      (effects (font (size 1.27 1.27)) hide)
-    )
-    (property "Manufacturer Part Number" "9774030243R" (id 5) (at 279.4 95.25 0)
-      (effects (font (size 1.27 1.27)) hide)
-    )
-    (property "Specification" "3.5mm length M2 threaded surface mounted steel standoffs " (id 6) (at 279.4 95.25 0)
-      (effects (font (size 1.27 1.27)) hide)
-    )
-  )
   (symbol (lib_id "power:GND") (at 357.505 569.595 90) (unit 1)
     (in_bom yes) (on_board yes)
@@
     (pin "1")
   )
-  (symbol (lib_id "Mechanical:MountingHole") (at 279.4 88.9 0) (unit 1)
-    (in_bom yes) (on_board yes)
-    (property "Reference" "H4" (id 0) (at 283.21 88.2649 0)
-      (effects (font (size 1.27 1.27)) (justify left))
-    )
-    (property "Value" "9774035243R" (id 1) (at 283.21 90.8049 0)
-      (effects (font (size 1.27 1.27)) (justify left))
-    )
-    (property "Footprint" "acheron_Hardware:9774035243R" (id 2) (at 279.4 88.9 0)
-      (effects (font (size 1.27 1.27)) hide)
-    )
-    (property "Datasheet" "~" (id 3) (at 279.4 88.9 0)
-      (effects (font (size 1.27 1.27)) hide)
-    )
-    (property "Manufacturer" "Wurth Elektronik" (id 4) (at 279.4 88.9 0)
-      (effects (font (size 1.27 1.27)) hide)
-    )
-    (property "Manufacturer Part Number" "9774030243R" (id 5) (at 279.4 88.9 0)
-      (effects (font (size 1.27 1.27)) hide)
-    )
-    (property "Specification" "3.5mm length M2 threaded surface mounted steel standoffs " (id 6) (at 279.4 88.9 0)
-      (effects (font (size 1.27 1.27)) hide)
-    )
-  )
   (sheet_instances
     (path "/" (page "1"))
@@
       (reference "H1") (unit 1) (value "9774035243R") (footprint "acheron_Hardware:9774035243R")
     )
-    (path "/50531c3d-35ad-4616-9dad-3d24868a8e99"
-      (reference "H2") (unit 1) (value "9774035243R") (footprint "acheron_Hardware:9774035243R")
-    )
-    (path "/072cb889-bb56-44ed-8362-4c25966840bb"
-      (reference "H3") (unit 1) (value "9774035243R") (footprint "acheron_Hardware:9774035243R")
-    )
-    (path "/ff60e663-e82b-4e68-b663-1e32f670ed8c"
-      (reference "H4") (unit 1) (value "9774035243R") (footprint "acheron_Hardware:9774035243R")
-    )
-    (path "/ef6e2432-2bff-4570-86a2-c6fe1895f389"
-      (reference "H5") (unit 1) (value "9774035243R") (footprint "acheron_Hardware:9774035243R")
-    )
-    (path "/2ff0b1f2-7f36-405d-8aa7-b31ef2214b4b"
-      (reference "H6") (unit 1) (value "9774035243R") (footprint "acheron_Hardware:9774035243R")
-    )
-    (path "/60827386-44a0-4288-9020-4b8850a133a3"
-      (reference "H7") (unit 1) (value "9774035243R") (footprint "acheron_Hardware:9774035243R")
-    )
-    (path "/d3b25a76-b015-4113-b74e-21ed415eb1e0"
-      (reference "H8") (unit 1) (value "9774035243R") (footprint "acheron_Hardware:9774035243R")
-    )
     (path "/888b62b0-e6e7-4413-9ebe-4d84f3056674"
