File: kb-lone.kicad_sch (KiCad schematic)
At the start: 468 parts, among them J1 TYPE-C-31-M12, J2 SM04B-SRSS-TB(LF)(SN), J3 SM04B-SRSS-TB(LF)(SN), J4 SSD1306, M1 RGB DB notch, Q1 DTC123JKAT146, SW1 K2-1187SQ-A4SW-06, SW10 F8, SW11 F9, SW12 F10, SW13 F11, SW14 F12, SW15 KNOB, SW16 GRV, SW17 1, SW18 2, SW19 3, SW2 ESC, SW20 4, SW21 5, SW22 6, SW23 7, SW24 8, SW25 9, SW26 0, SW27 MINUS, SW28 EQUAL, SW29 BSPC, SW3 F1, SW30 N/A, SW31 TAB, SW32 Q, SW33 W, SW34 E, SW35 R, SW36 T, SW37 Y, SW38 U, SW39 I, SW4 F2, SW40 O, SW41 P, SW42 LBRKT, SW43 RBRKT, SW44 BSLS, SW45 N/A, SW46 CAPS, SW47 A, SW48 S, SW49 D, SW5 F3, SW50 F, SW51 G, SW52 H, SW53 J, SW54 K, SW55 L, SW56 COLON, SW57 QUOTE, SW58 ENTER, SW59 PGUP, SW6 F4, SW60 LSHFT, SW61 Z, SW62 X, SW63 C, SW64 V, SW65 B, SW66 N, SW67 M, SW68 COMMA, SW69 DOT, SW7 F5, SW70 SLSH, SW71 RSHFT, SW72 UP, SW73 PGDN, SW74 LCTRL, SW75 WIN, SW76 LALT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

Commit message: fix edge cuts
Parts:
- C1, C17, C18, C3: Manufacturer (none) -> YAGEO; Manufacturer Part Number (none) -> CC0805KRX7R9BB104; Specification MLCC 10V or more -> 50V 10% X7R 0805; Vendor Part Number (none) -> ELESKU 302010165
- C10, C9: Manufacturer (none) -> Murata; Manufacturer Part Number (none) -> GRM1555C1H150JA01D; Specification MLCC 10V or more -> 50V 5% 0402; Vendor Part Number (none) -> ELESKU 302010041
- C100, C14, C15, C19, C20, C21, C22, C23, C24, C25, C26, C27, C28, C29, C30, C31, C32, C33, C34, C35, C36, C37, C38, C39, C40, C41, C42, C43, C44, C45, C46, C47, C48, C49, C50, C51, C52, C53, C54, C55, C56, C57, C58, C59, C6, C60, C61, C62, C63, C64, C65, C66, C67, C68, C69, C7, C70, C71, C72, C73, C74, C75, C76, C77, C78, C8, C80, C81, C82, C83, C84, C85, C86, C87, C88, C89, C90, C91, C92, C93, C94, C95, C96, C97, C98, C99: Manufacturer (none) -> YAGEO; Manufacturer Part Number (none) -> CC0402KRX7R8BB104; Specification MLCC 10V or more -> 25V 10% X7R; Vendor Part Number (none) -> ELESKU 302010024
- C11, C16: Manufacturer (none) -> Murata; Manufacturer Part Number (none) -> GRM155R60J475KE96D; Specification MLCC 10V or more -> 6.3V 10% X5R 0402; Vendor Part Number (none) -> ELESZ GRM155R60J475KE96D
- C12: Manufacturer (none) -> YAGEO; Manufacturer Part Number (none) -> CC0402KRX7R9BB103; Specification MLCC 10V or more -> 50V 10% X7R 0402; Vendor Part Number (none) -> ELESKU 302010006
- C13: Manufacturer (none) -> AVX; Manufacturer Part Number (none) -> TAJA106K016RNJ; Specification Tantallum CASEA capacitor rated 10V or more -> 16V 10% tantallum 3216 (CASE-A); Vendor Part Number (none) -> ELESKU 302020002
- C2: Manufacturer (none) -> Samsung; Manufacturer Part Number (none) -> CL21B105KOFNNNE; Specification MLCC 10V or more -> 10% 16V X7R 0805; Vendor Part Number (none) -> ELESZ CL21B105KOFNNNE
- C4, C5: Manufacturer (none) -> YAGEO; Manufacturer Part Number (none) -> CC0805KKX7R8BB105; Specification MLCC 10V or more -> 10% 25V X7R 0805; Vendor Part Number (none) -> ELESKU 302010179
- C79:   (none) -> 25V 10% X7R; Manufacturer (none) -> YAGEO; Manufacturer Part Number (none) -> CC0402KRX7R8BB104; Specification MLCC 10V or more -> (none); Vendor Part Number (none) -> ELESKU 302010024
- D1: Manufacturer (none) -> Microdiode Electronics; Manufacturer Part Number (none) -> 1N4148W; Specification Small signal switching diode -> Small-signal switching diodes; Vendor Part Number (none) -> LCSC C84367 / ELESKU 1N4148W-7-F
- D10, D11, D12, D13, D14, D15, D16, D17, D18, D19, D20, D21, D22, D23, D24, D25, D26, D27, D28, D29, D3, D30, D31, D32, D33, D34, D35, D36, D37, D38, D39, D4, D40, D41, D42, D43, D44, D45, D46, D47, D48, D49, D5, D50, D51, D52, D53, D54, D55, D56, D57, D58, D59, D6, D60, D61, D62, D63, D64, D65, D66, D67, D68, D69, D7, D70, D71, D72, D73, D74, D75, D76, D77, D78, D79, D8, D80, D81, D82, D83, D84, D9: Manufacturer (none) -> Microdiode Electronics; Manufacturer Part Number (none) -> 1N4148W; Vendor Part Number (none) -> LCSC C84367 / ELESKU 1N4148W-7-F
- D2: Vendor Part Number LCSC C114257 -> LCSC C114257 / ELESZ RB060M-60
- F1: Vendor Part Number LCSC C69691 -> LCSC C69691 / ELESKU mSMD110-16V
- H2, H3, H4, H5: value MountingHole -> 9774035243R; Manufacturer (none) -> Wurth Elektronik; Manufacturer Part Number (none) -> 9774030243R; Specification (none) -> 3.5mm length M2 threaded surface mounted steel standoffs
- J1: Vendor Part Number LCSC C165948 -> ELESZ TYPE-C-31-M-12 / LCSC C165948
- Q1: Vendor Part Number LCSC C111724 -> ELESZ DTC123JKAT146 / LCSC C111724
- R1, R2: Manufacturer (none) -> YAGEO; Manufacturer Part Number (none) -> RC0805FR-075K1L; Specification (none) -> 1% 1/8W 0805; Vendor Part Number (none) -> ELESKU 301012180
- R10, R9: Manufacturer (none) -> YAGEO; Manufacturer Part Number (none) -> RC0402JR-074K7L; Specification (none) -> 5% 1/16W 0402; Vendor Part Number (none) -> ELESKU 301012026
- R13: Manufacturer (none) -> YAGEO; Manufacturer Part Number (none) -> RC0402FR-071K5L; Specification (none) -> 1% 1/16W 0402; Vendor Part Number (none) -> ELESKU 301011987
- R14, R8: Manufacturer (none) -> YAGEO; Manufacturer Part Number (none) -> RC0805FR-0710KL; Specification (none) -> 1% 1/8W 0805; Vendor Part Number (none) -> ELESKU 301012152
- R15, R16, R17, R18, R19, R20, R21, R22, R23, R24, R25, R26, R27, R28, R29, R30, R31, R32, R33, R34, R35, R36, R37, R38, R39, R40, R41, R42, R43, R44, R45, R46, R47, R48, R49, R50, R51, R52, R53, R54, R55, R56, R57, R58, R59, R60, R61, R62, R63, R64, R65, R66, R67, R68, R69, R70, R71, R72, R73, R74, R75, R76, R77, R78, R79, R80, R81, R82, R83, R84, R85, R86, R87, R88, R89, R90, R91, R92, R93, R94, R95, R96: Manufacturer (none) -> Walsin; Manufacturer Part Number (none) -> WR04X5R1JTL; Specification (none) -> 1% 1/16W 0402; Vendor Part Number (none) -> ELESZ WR04X5R1JTL
- R3: Manufacturer (none) -> YAGEO; Manufacturer Part Number (none) -> RC0805JR-07100RL; Specification (none) -> 1% 1/8W 0805; Vendor Part Number (none) -> ELESKU 301010319
- R4: Manufacturer (none) -> YAGEO; Manufacturer Part Number (none) -> RC0805FR-07330KL; Specification (none) -> 1% 1/8W 0805; Vendor Part Number (none) -> ELESZ RC0805FR-07330KL
- R5: Manufacturer (none) -> YAGEO; Manufacturer Part Number (none) -> RC0805FR-071ML; Specification (none) -> 1% 1/8W 0805; Vendor Part Number (none) -> ELESZ RC0805FR-071ML
- R6, R7: Manufacturer (none) -> YAGEO; Manufacturer Part Number (none) -> RC0805FR-07100KL; Specification (none) -> 1% 1/8W 0805; Vendor Part Number (none) -> ELESKU 301012150
- Y1: Vendor Part Number LCSC C403948 -> ELESZ TAXM8M4RFDCET2T / LCSC C403948

Commit message: daughter board
Parts:
- removed F1: mSMD110-16V, Fuse:Fuse_1812_4532Metric, symbol Device:Fuse
- removed FB2: CBW201209U121T, Inductor_SMD:L_0805_2012Metric, symbol Device:Ferrite_Bead_Small
- removed H9: MountingHole, acheron_MountingHoles:MountingHole_2.5x4.0mm, symbol Mechanical:MountingHole_Pad
- removed J1: TYPE-C-31-M12, acheron_Connectors:TYPE-C-31-M-12, symbol acheronSymbols:USB_C_16_pin
- removed R1, R2: 5.1k, Resistor_SMD:R_0805_2012Metric, symbol Device:R_Small
- removed U1: USBLC6-2SC6, Package_TO_SOT_SMD:SOT-23-6, symbol Power_Protection:USBLC6-2SC6
Connections:
- no-connect marks 17 -> 15
Other:
- note added: "Unified-Daughterboard"

Commit message: layout
Parts:
- removed C47: 100n, apollo87h_kicad_library:C_0402_1005Metric_1, symbol Device:C_Small
- removed D113: SK6812MINI-E, acheron_Components:SK6812MINI_3535_6028_3.2x2.8mm_Round, symbol acheron_Symbols:SK6812MINI-E
- removed D16, D31: 1N4148W, acheron_Components:D_SOD-123, symbol Device:D
- removed R43: 5.1R, apollo87h_kicad_library:R_0402_1005Metric_1, symbol Device:R_Small
- removed SW15: KNOB, acheron_MXA:MXA100, symbol acheronSymbols:Mechanical_Switch
- removed SW30: N/A, acheron_MXH_MetalRings:MX100H, symbol acheronSymbols:Mechanical_Switch
Connections:
- net at D128.4 (DIN): now also D112.2 (DOUT)
